File: hw/ECE445L_Lab7/Lab7_LeftAudio.kicad_sch (KiCad schematic)
At the start: 39 parts, among them IC2 TLV5616, Q2 PZT2222A, Q3 PZT2222A, Q4 PZT2222A, Q5 PZT2222A, Q6 PZT2222A, Q7 PZT2222A, U3 OPA2350, U4 OPA2350, U5 OPA2350, U6 OPA2350

Commit message: Updated hardware schematic
Parts:
- removed C1, C2, C4, C5, C6, C7: C, Capacitor_SMD:C_0805_2012Metric, symbol ECE445L:C
- removed C10, C16, C8, C9: .1u, Capacitor_SMD:C_0805_2012Metric, symbol ECE445L:C
- removed C3: 0.1u, ECE445L:C_Axial_200mil, symbol ECE445L:C
- removed IC2: TLV5616, ECE445L:DIP-8_W7.62mm_LongPads, symbol ECE445L:TLV5616
- removed Q2, Q3, Q4, Q5, Q6, Q7: PZT2222A, Package_TO_SOT_SMD:SOT-223-3_TabPin2, symbol Transistor_BJT:PZT2222A
- removed R1, R10, R14, R15, R16, R2, R9: R, Resistor_SMD:R_0805_2012Metric, symbol Device:R
- removed R11, R17, R7: 20k, Resistor_SMD:R_0805_2012Metric, symbol Device:R
- removed R12, R13, R18, R19, R20, R6, R8: 10k, Resistor_SMD:R_0805_2012Metric, symbol Device:R
- removed U3, U4, U5, U6: OPA2350, ECE445L:DIP-8_W7.62mm_LongPads, symbol ECE445L:OPA2350
- added C28, C29, C30, C31, C34, C35: C, Capacitor_SMD:C_0805_2012Metric, symbol ECE445L:C
- added C32, C33, C36: .1u, Capacitor_SMD:C_0805_2012Metric, symbol ECE445L:C
- added C38: 0.1u, ECE445L:C_Axial_200mil, symbol ECE445L:C
- added Q10, Q11, Q12, Q13, Q14, Q9: PZT2222A, Package_TO_SOT_SMD:SOT-223-3_TabPin2, symbol Transistor_BJT:PZT2222A
- added R23, R26, R27, R28, R29, R36, R37: R, Resistor_SMD:R_0805_2012Metric, symbol Device:R
- added R30, R31, R38: 20k, Resistor_SMD:R_0805_2012Metric, symbol Device:R
- added R32, R33, R34, R35, R39, R40, R41: 10k, Resistor_SMD:R_0805_2012Metric, symbol Device:R
- added U10, U6, U8, U9: OPA2350, ECE445L:DIP-8_W7.62mm_LongPads, symbol ECE445L:OPA2350
- added U4: TLV5616, ECE445L:DIP-8_W7.62mm_LongPads, symbol ECE445L:TLV5616
Connections:
- net +3V3: now also C32.2, C33.2, C36.2, C38.1, R28.2, R36.2, U10.8 (V+), U4.8 (VDD), U8.8 (V+), U9.8 (V+)
- net GND: now also C31.2, C32.1, C33.1, C35.1, C36.1, C38.2, Q10.3 (E), Q11.3 (E), Q12.3 (E), Q13.3 (E), Q14.3 (E), Q9.3 (E), R29.1, R37.1, U10.4 (V-), U4.3 (~{CS}), U4.5 (AGND), U8.4 (V-), U9.4 (V-)
- net PD0: now also Q12.1 (B)
- net PD1: now also Q10.1 (B)
- net PD2: now also Q14.1 (B)
- net PD3: now also Q13.1 (B)
- net PD4: now also Q11.1 (B)
- net PD5: now also Q9.1 (B)
- net R_Bass: now also U10.6 (-), U10.7, U6.5 (+), U8.6 (-), U8.7, U9.6 (-), U9.7
- net VRef: now also U4.6 (REF)
- net Vin: now also C28.1, C34.1, R23.2, U4.7 (OUT)
- new net: C29.1, R35.2, U9.1, U9.5 (+)
- new net: C29.2, R23.1, R27.1
- new net: R26.1, R34.2, U8.1, U8.5 (+)
- new net: R30.1, R32.2, R34.1, U8.2 (-)
- new net: C30.2, R28.1, R29.2, U8.3 (+)
- new net: Q12.2 (C), R33.1
- new net: R38.1, R39.2, R40.1, U10.2 (-)
- new net: R40.2, R41.1, U10.1
- new net: C28.2, C30.1, R26.2
- new net: Q11.2 (C), R32.1
- new net: Q9.2 (C), R30.2
- new net: R36.1, R37.2
- new net: Q13.2 (C), R38.2
- new net: C35.2, R41.2, U10.5 (+)
- new net: C34.2, U10.3 (+)
- new net: C31.1, R27.2, U9.3 (+)
- new net: Q14.2 (C), R39.1
- new net: R31.1, R33.2, R35.1, U9.2 (-)
- new net: Q10.2 (C), R31.2
- new net ESP_GPIO3: U4.1 (DIN)
- new net ESP_GPIO4: U4.2 (SCLK)
- new net ESP_GPIO5: U4.4 (FS)
- new net R_Out: U6.6 (-), U6.7

Commit message: More Updates to hardware
Parts:
- renumbered U9 to U11, U10 to U12, U8 to U13, U6 to U14, U4 to U6
Connections:
- net Vin: no longer R23.2, U6.7 (OUT)
- new net Vin_R: R23.2, U6.7 (OUT)
Changed lines of the file:
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@@
 		)
 	)
-	(global_label "Vin"
+	(global_label "Vin_R"
 		(shape input)
 		(at 21.59 151.765 180)
@@
 		)
 		(property "Intersheetrefs" "${INTERSHEET_REFS}"
-			(at 15.7624 151.765 0)
+			(at 13.5248 151.765 0)
 			(effects
 				(font
@@
 		)
 	)
-	(global_label "Vin"
+	(global_label "Vin_R"
 		(shape input)
 		(at 260.985 134.62 0)
@@
 		)
 		(property "Intersheetrefs" "${INTERSHEET_REFS}"
-			(at 266.8126 134.62 0)
+			(at 269.0502 134.62 0)
 			(effects
 				(font
@@
 		(dnp no)
 		(fields_autoplaced yes)
-		(property "Reference" "U8"
+		(property "Reference" "U13"
 			(at 61.595 30.48 0)
 			(effects
@@
 			(project "ECE445L_Lab7"
 				(path "/69b823fd-c065-40ff-9bb9-c5835555f3eb/8e43ed7d-abc3-4582-a9a6-069be8f9db2b"
-					(reference "U8")
+					(reference "U13")
 					(unit 1)
 				)
@@
 		(dnp no)
 		(fields_autoplaced yes)
-		(property "Reference" "U8"
+		(property "Reference" "U13"
 			(at 90.17 33.02 0)
 			(effects
@@
 			(project "ECE445L_Lab7"
 				(path "/69b823fd-c065-40ff-9bb9-c5835555f3eb/8e43ed7d-abc3-4582-a9a6-069be8f9db2b"
-					(reference "U8")
+					(reference "U13")
 					(unit 2)
 				)
@@
 		(dnp no)
 		(fields_autoplaced yes)
-		(property "Reference" "U4"
+		(property "Reference" "U6"
 			(at 225.425 124.46 0)
 			(effects
@@
 			(project "ECE445L_Lab7"
 				(path "/69b823fd-c065-40ff-9bb9-c5835555f3eb/8e43ed7d-abc3-4582-a9a6-069be8f9db2b"
-					(reference "U4")
+					(reference "U6")
 					(unit 1)
 				)
@@
 		(dnp no)
 		(fields_autoplaced yes)
-		(property "Reference" "U10"
+		(property "Reference" "U12"
 			(at 180.975 71.12 0)
 			(effects
@@
 			(project "ECE445L_Lab7"
 				(path "/69b823fd-c065-40ff-9bb9-c5835555f3eb/8e43ed7d-abc3-4582-a9a6-069be8f9db2b"
-					(reference "U10")
+					(reference "U12")
 					(unit 2)
 				)
@@
 		(dnp no)
 		(fields_autoplaced yes)
-		(property "Reference" "U10"
-			(at 174.625 111.1249 0)
+		(property "Reference" "U12"
+			(at 173.99 111.1249 0)
 			(effects
 				(font
@@
 		)
 		(property "Value" "OPA2350"
-			(at 174.625 113.6649 0)
+			(at 173.99 113.6649 0)
 			(effects
 				(font
@@
 			(project "ECE445L_Lab7"
 				(path "/69b823fd-c065-40ff-9bb9-c5835555f3eb/8e43ed7d-abc3-4582-a9a6-069be8f9db2b"
-					(reference "U10")
+					(reference "U12")
 					(unit 3)
 				)
@@
 		(dnp no)
 		(fields_autoplaced yes)
-		(property "Reference" "U10"
+		(property "Reference" "U12"
 			(at 139.065 68.58 0)
 			(effects
@@
 			(project "ECE445L_Lab7"
 				(path "/69b823fd-c065-40ff-9bb9-c5835555f3eb/8e43ed7d-abc3-4582-a9a6-069be8f9db2b"
-					(reference "U10")
+					(reference "U12")
 					(unit 1)
 				)
@@
 		(dnp no)
 		(fields_autoplaced yes)
-		(property "Reference" "U6"
+		(property "Reference" "U14"
 			(at 165.735 26.67 0)
 			(effects
@@
 			(project "ECE445L_Lab7"
 				(path "/69b823fd-c065-40ff-9bb9-c5835555f3eb/8e43ed7d-abc3-4582-a9a6-069be8f9db2b"
-					(reference "U6")
+					(reference "U14")
 					(unit 2)
 				)
@@
 		(dnp no)
 		(fields_autoplaced yes)
-		(property "Reference" "U9"
-			(at 90.805 146.685 0)
+		(property "Reference" "U11"
+			(at 90.805 147.32 0)
 			(effects
 				(font
@@
 		)
 		(property "Value" "OPA2350"
-			(at 90.805 149.225 0)
+			(at 90.805 149.86 0)
 			(effects
 				(font
@@
 			(project "ECE445L_Lab7"
 				(path "/69b823fd-c065-40ff-9bb9-c5835555f3eb/8e43ed7d-abc3-4582-a9a6-069be8f9db2b"
-					(reference "U9")
+					(reference "U11")
 					(unit 2)
 				)
@@
 		(dnp no)
 		(fields_autoplaced yes)
-		(property "Reference" "U9"
-			(at 62.23 144.145 0)
+		(property "Reference" "U11"
+			(at 62.23 144.78 0)
 			(effects
 				(font
@@
 		)
 		(property "Value" "OPA2350"
-			(at 62.23 146.685 0)
+			(at 62.23 147.32 0)
 			(effects
 				(font
@@
 			(project "ECE445L_Lab7"
 				(path "/69b823fd-c065-40ff-9bb9-c5835555f3eb/8e43ed7d-abc3-4582-a9a6-069be8f9db2b"
-					(reference "U9")
+					(reference "U11")
 					(unit 1)
 				)
@@
 		(dnp no)
 		(fields_autoplaced yes)
-		(property "Reference" "U9"
-			(at 94.615 180.3399 0)
+		(property "Reference" "U11"
+			(at 93.98 180.3399 0)
 			(effects
 				(font
@@
 		)
 		(property "Value" "OPA2350"
-			(at 94.615 182.8799 0)
+			(at 93.98 182.8799 0)
 			(effects
 				(font
@@
 			(project "ECE445L_Lab7"
 				(path "/69b823fd-c065-40ff-9bb9-c5835555f3eb/8e43ed7d-abc3-4582-a9a6-069be8f9db2b"
-					(reference "U9")
+					(reference "U11")
 					(unit 3)
 				)
@@
 		(dnp no)
 		(fields_autoplaced yes)
-		(property "Reference" "U8"
+		(property "Reference" "U13"
 			(at 104.14 26.6699 0)
 			(effects
@@
 			(project "ECE445L_Lab7"
 				(path "/69b823fd-c065-40ff-9bb9-c5835555f3eb/8e43ed7d-abc3-4582-a9a6-069be8f9db2b"
-					(reference "U8")
+					(reference "U13")
 					(unit 3)
 				)
