File: hw/ECE445L_Lab7/Lab7_LeftAudio.kicad_sch (KiCad schematic)
At the start: 69 parts, among them Q10 MMBF170, Q11 MMBF170, Q12 MMBF170, Q13 MMBF170, Q14 MMBF170, Q15 MMBF170, Q16 MMBF170, Q17 MMBF170, Q18 MMBF170, U11 OPA2350, U12 OPA2350, U13 OPA2350, U14 OPA2350, U15 TLV5616

Commit message: Final PCB commit
Parts:
- removed Q16, Q17, Q18: MMBF170, Package_TO_SOT_SMD:SOT-23-3, symbol Transistor_BJT:PZT2222A
- removed R111, R112, R113: 2k, Resistor_SMD:R_0603_1608Metric_Pad0.98x0.95mm_HandSolder, symbol Device:R
- removed R63, R65, R66, R67, R69: 100k, Resistor_SMD:R_0603_1608Metric_Pad0.98x0.95mm_HandSolder, symbol Device:R
- removed R68: 75K, Resistor_SMD:R_0603_1608Metric_Pad0.98x0.95mm_HandSolder, symbol Device:R
- Q10: renamed from Q13; footprint Package_TO_SOT_SMD:SOT-23-3 -> Package_TO_SOT_SMD:SOT-23; symbol Transistor_BJT:PZT2222A -> Transistor_FET:MMBF170
- Q11: renamed from Q14; footprint Package_TO_SOT_SMD:SOT-23-3 -> Package_TO_SOT_SMD:SOT-23; symbol Transistor_BJT:PZT2222A -> Transistor_FET:MMBF170
- Q12: renamed from Q15; footprint Package_TO_SOT_SMD:SOT-23-3 -> Package_TO_SOT_SMD:SOT-23; symbol Transistor_BJT:PZT2222A -> Transistor_FET:MMBF170
- Q7: renamed from Q10; footprint Package_TO_SOT_SMD:SOT-23-3 -> Package_TO_SOT_SMD:SOT-23; symbol Transistor_BJT:PZT2222A -> Transistor_FET:MMBF170
- Q8: renamed from Q11; footprint Package_TO_SOT_SMD:SOT-23-3 -> Package_TO_SOT_SMD:SOT-23; symbol Transistor_BJT:PZT2222A -> Transistor_FET:MMBF170
- Q9: renamed from Q12; footprint Package_TO_SOT_SMD:SOT-23-3 -> Package_TO_SOT_SMD:SOT-23; symbol Transistor_BJT:PZT2222A -> Transistor_FET:MMBF170
- R47: renamed from R42; value 100k -> 184k
- R48: renamed from R43; value 100k -> 68.8k
- R49: renamed from R44; value 20k -> 40k
- R50: renamed from R45; value 20k -> 40k
- R51: renamed from R46; value 10k -> 30k
- R52: renamed from R47; value 10k -> 30k
- R58: renamed from R50; value 100k -> 184k
- R59: renamed from R51; value 100k -> 68.8k
- R60: renamed from R52; value 20k -> 40k
- R61: renamed from R53; value 10k -> 30k
- R72: renamed from R64; value 100k -> 50k
- renumbered C27 to C16, C28 to C17, C29 to C18, C30 to C19, C31 to C20, C32 to C21, C33 to C22, C34 to C23, C35 to C24, C36 to C25, C37 to C26, C38 to C27, R39 to R42, R40 to R43, R109 to R44, R107 to R45, R41 to R46, R48 to R53, R49 to R54, R110 to R55, R108 to R56, R105 to R57, R54 to R62, R106 to R63, R55 to R64, R58 to R65, R56 to R66, R57 to R67, R59 to R68, R60 to R69, R61 to R70, R62 to R71, TP8 to TP10, TP9 to TP11, TP10 to TP12, U11 to U10, U12 to U11, U13 to U12, U14 to U13, U15 to U14
Connections:
- net GND: now also Q10.2 (S), Q11.2 (S), Q12.2 (S), Q7.2 (S), Q8.2 (S), Q9.2 (S); no longer Q10.3 (E), Q11.3 (E), Q12.3 (E), Q7.3 (E), Q8.3 (E), Q9.3 (E)
- net at R60.2: now also Q11.3 (D); no longer Q11.2 (C)
- net at R50.2: now also Q8.3 (D); no longer Q8.2 (C)
- net at R51.2: now also Q9.3 (D); no longer Q9.2 (C)
- net at R49.2: now also Q7.3 (D); no longer Q7.2 (C)
- net at C26.2, R70.1, R71.2: now also U13.5 (+); no longer R72.1
- net at R52.2: now also Q10.3 (D); no longer Q10.2 (C)
- net at R61.2: now also Q12.3 (D); no longer Q12.2 (C)
- net L_AudioOut renamed L_AudioBuf
- net L_AudioBuf: now also R72.1
Other:
- moved on the sheet: C26, R66, R67, R68, R70, R71, R72, U13A, U13B
