File: hw/ECE445L_Lab7/Lab7_analog.kicad_sch (KiCad schematic)
At the start: 39 parts, among them IC2 TLV5616, Q2 PZT2222A, Q3 PZT2222A, Q4 PZT2222A, Q5 PZT2222A, Q6 PZT2222A, Q7 PZT2222A, U3 OPA2350, U4 OPA2350, U5 OPA2350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

Commit message: More Updates to hardware
Parts:
- renumbered U4 to U10, U6 to U14, IC2 to U5, U3 to U8, U5 to U9
Connections:
- net Vin: no longer R1.2, U5.7 (OUT)
- new net Vin_L: R1.2, U5.7 (OUT)
Changed lines of the file:
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@@
 		)
 	)
-	(global_label "Vin"
+	(global_label "Vin_L"
 		(shape input)
 		(at 260.985 134.62 0)
@@
 		)
 		(property "Intersheetrefs" "${INTERSHEET_REFS}"
-			(at 266.8126 134.62 0)
+			(at 268.8083 134.62 0)
 			(effects
 				(font
@@
 		)
 	)
-	(global_label "Vin"
+	(global_label "Vin_L"
 		(shape input)
 		(at 21.59 151.765 180)
@@
 		)
 		(property "Intersheetrefs" "${INTERSHEET_REFS}"
-			(at 15.7624 151.765 0)
+			(at 13.7667 151.765 0)
 			(effects
 				(font
@@
 		(dnp no)
 		(fields_autoplaced yes)
-		(property "Reference" "U3"
-			(at 90.805 146.685 0)
+		(property "Reference" "U8"
+			(at 90.805 147.32 0)
 			(effects
 				(font
@@
 		)
 		(property "Value" "OPA2350"
-			(at 90.805 149.225 0)
+			(at 90.805 149.86 0)
 			(effects
 				(font
@@
 			(project ""
 				(path "/69b823fd-c065-40ff-9bb9-c5835555f3eb/9e7b1dfa-492f-407a-9f72-cee77954c346"
-					(reference "U3")
+					(reference "U8")
 					(unit 2)
 				)
@@
 		(dnp no)
 		(fields_autoplaced yes)
-		(property "Reference" "IC2"
+		(property "Reference" "U5"
 			(at 225.425 124.46 0)
 			(effects
@@
 			(project "ECE445L_Lab7"
 				(path "/69b823fd-c065-40ff-9bb9-c5835555f3eb/9e7b1dfa-492f-407a-9f72-cee77954c346"
-					(reference "IC2")
+					(reference "U5")
 					(unit 1)
 				)
@@
 		(dnp no)
 		(fields_autoplaced yes)
-		(property "Reference" "U6"
+		(property "Reference" "U14"
 			(at 165.735 26.67 0)
 			(effects
@@
 			(project ""
 				(path "/69b823fd-c065-40ff-9bb9-c5835555f3eb/9e7b1dfa-492f-407a-9f72-cee77954c346"
-					(reference "U6")
+					(reference "U14")
 					(unit 1)
 				)
@@
 		(dnp no)
 		(fields_autoplaced yes)
-		(property "Reference" "U5"
+		(property "Reference" "U9"
 			(at 180.975 71.12 0)
 			(effects
@@
 			(project ""
 				(path "/69b823fd-c065-40ff-9bb9-c5835555f3eb/9e7b1dfa-492f-407a-9f72-cee77954c346"
-					(reference "U5")
+					(reference "U9")
 					(unit 2)
 				)
@@
 		(dnp no)
 		(fields_autoplaced yes)
-		(property "Reference" "U5"
+		(property "Reference" "U9"
 			(at 139.065 68.58 0)
 			(effects
@@
 			(project ""
 				(path "/69b823fd-c065-40ff-9bb9-c5835555f3eb/9e7b1dfa-492f-407a-9f72-cee77954c346"
-					(reference "U5")
+					(reference "U9")
 					(unit 1)
 				)
@@
 		(dnp no)
 		(fields_autoplaced yes)
-		(property "Reference" "U5"
-			(at 174.625 111.1249 0)
+		(property "Reference" "U9"
+			(at 173.99 111.1249 0)
 			(effects
 				(font
@@
 		)
 		(property "Value" "OPA2350"
-			(at 174.625 113.6649 0)
+			(at 173.99 113.6649 0)
 			(effects
 				(font
@@
 			(project ""
 				(path "/69b823fd-c065-40ff-9bb9-c5835555f3eb/9e7b1dfa-492f-407a-9f72-cee77954c346"
-					(reference "U5")
+					(reference "U9")
 					(unit 3)
 				)
@@
 		(dnp no)
 		(fields_autoplaced yes)
-		(property "Reference" "U4"
+		(property "Reference" "U10"
 			(at 104.14 26.6699 0)
 			(effects
@@
 			(project "ECE445L_Lab7"
 				(path "/69b823fd-c065-40ff-9bb9-c5835555f3eb/9e7b1dfa-492f-407a-9f72-cee77954c346"
-					(reference "U4")
+					(reference "U10")
 					(unit 3)
 				)
@@
 		(dnp no)
 		(fields_autoplaced yes)
-		(property "Reference" "U4"
+		(property "Reference" "U10"
 			(at 61.595 30.48 0)
 			(effects
@@
 			(project "ECE445L_Lab7"
 				(path "/69b823fd-c065-40ff-9bb9-c5835555f3eb/9e7b1dfa-492f-407a-9f72-cee77954c346"
-					(reference "U4")
+					(reference "U10")
 					(unit 1)
 				)
@@
 		(dnp no)
 		(fields_autoplaced yes)
-		(property "Reference" "U4"
+		(property "Reference" "U10"
 			(at 90.17 33.02 0)
 			(effects
@@
 			(project "ECE445L_Lab7"
 				(path "/69b823fd-c065-40ff-9bb9-c5835555f3eb/9e7b1dfa-492f-407a-9f72-cee77954c346"
-					(reference "U4")
+					(reference "U10")
 					(unit 2)
 				)
@@
 		(dnp no)
 		(fields_autoplaced yes)
-		(property "Reference" "U3"
-			(at 94.615 180.3399 0)
+		(property "Reference" "U8"
+			(at 93.98 180.3399 0)
 			(effects
 				(font
@@
 		)
 		(property "Value" "OPA2350"
-			(at 94.615 182.8799 0)
+			(at 93.98 182.8799 0)
 			(effects
 				(font
@@
 			(project ""
 				(path "/69b823fd-c065-40ff-9bb9-c5835555f3eb/9e7b1dfa-492f-407a-9f72-cee77954c346"
-					(reference "U3")
+					(reference "U8")
 					(unit 3)
 				)
@@
 		(dnp no)
 		(fields_autoplaced yes)
-		(property "Reference" "U6"
+		(property "Reference" "U14"
 			(at 209.55 29.8449 0)
 			(effects
@@
 			(project ""
 				(path "/69b823fd-c065-40ff-9bb9-c5835555f3eb/9e7b1dfa-492f-407a-9f72-cee77954c346"
-					(reference "U6")
+					(reference "U14")
 					(unit 3)
 				)
@@
 		(dnp no)
 		(fields_autoplaced yes)
-		(property "Reference" "U3"
-			(at 62.23 144.145 0)
+		(property "Reference" "U8"
+			(at 62.23 144.78 0)
 			(effects
 				(font
@@
 		)
 		(property "Value" "OPA2350"
-			(at 62.23 146.685 0)
+			(at 62.23 147.32 0)
 			(effects
 				(font
@@
 			(project ""
 				(path "/69b823fd-c065-40ff-9bb9-c5835555f3eb/9e7b1dfa-492f-407a-9f72-cee77954c346"
-					(reference "U3")
+					(reference "U8")
 					(unit 1)
 				)
