File: hw/ECE445L_Lab7/ECE445L_Lab7.kicad_pcb (KiCad board)
At the start: 2 copper layers, 115 x 94 mm, 18 parts, among them Q1 IRLD024PBF, SW1 UP, SW2 DOWN, SW3 LEFT, SW4 RIGHT, SW5 MODE, U1 EK-TM4C123GXL, U2 Adafruit ST7735R, U3 ESP8266-01/ESP-01

Commit message: Made changers to the schematic, updated bom, and created priliminary layout for the PCB. Ready for 7B Prep!
Parts:
- removed D1: 1N914, ECE445L:D_P6.35mm_Horizontal
- removed LS1: Speaker, ECE445L:PinHeader_1x02_P2.54mm_Vertical
- added C10: 10pF C0G, Capacitor_SMD:C_0603_1608Metric, F.Cu at (222.6, 142.1)
- added C11: 1uF, Capacitor_SMD:C_0603_1608Metric, F.Cu at (218.3, 134.2)
- added C12: 0.1u, Capacitor_SMD:C_0603_1608Metric, F.Cu at (160.5, 85.6)
- added C13: 10u, Capacitor_SMD:C_0805_2012Metric, B.Cu at (169.2, 84.1)
- added C14: 0.1u, Capacitor_SMD:C_0603_1608Metric, F.Cu at (164.1, 85.6)
- added C15: 27n, Capacitor_SMD:C_0603_1608Metric, F.Cu at (218.2, 82.8)
- added C16: 27n, Capacitor_SMD:C_0603_1608Metric, B.Cu at (215.1, 89.4)
- added C17: 10n, Capacitor_SMD:C_0603_1608Metric, F.Cu at (220.5, 99.6)
- added C18: 3.5n, Capacitor_SMD:C_0603_1608Metric, F.Cu at (203.2, 93.2)
- added C19: 1.2n, Capacitor_SMD:C_0603_1608Metric, F.Cu at (221.2, 103.1)
- added C20: 1.2n, Capacitor_SMD:C_0603_1608Metric, F.Cu at (218.2, 110.0)
- added C21: 10u, Capacitor_SMD:C_0805_2012Metric, F.Cu at (195.6, 96.3)
- added C22: 0.1u, Capacitor_SMD:C_0603_1608Metric, F.Cu at (203.5, 78.0)
- added C23: 0.1u, Capacitor_SMD:C_0603_1608Metric, B.Cu at (207.8, 106.9)
- added C24: 0.1u, Capacitor_SMD:C_0603_1608Metric, F.Cu at (206.0, 91.7)
- added C25: 0.1u, Capacitor_SMD:C_0603_1608Metric, B.Cu at (204.0, 107.2)
- added C26: 0.1u, Capacitor_SMD:C_0603_1608Metric, F.Cu at (225.3, 104.1)
- added C27: 27n, Capacitor_SMD:C_0603_1608Metric, F.Cu at (261.9, 112.8)
- added C28: 27n, Capacitor_SMD:C_0603_1608Metric, B.Cu at (264.9, 106.2)
- added C29: 10n, Capacitor_SMD:C_0603_1608Metric, F.Cu at (259.6, 96.0)
- added C3: 0.1uF, Capacitor_SMD:C_0603_1608Metric, F.Cu at (203.3, 130.9)
- added C30: 3.5n, Capacitor_SMD:C_0603_1608Metric, F.Cu at (276.9, 102.4)
- added C31: 1.2n, Capacitor_SMD:C_0603_1608Metric, F.Cu at (258.8, 92.4)
- added C32: 1.2n, Capacitor_SMD:C_0603_1608Metric, F.Cu at (261.9, 85.6)
- added C33: 0.1u, Capacitor_SMD:C_0603_1608Metric, F.Cu at (276.6, 117.6)
- added C34: 0.1u, Capacitor_SMD:C_0603_1608Metric, B.Cu at (276.1, 88.4)
- added C35: 0.1u, Capacitor_SMD:C_0603_1608Metric, F.Cu at (274.1, 103.9)
- added C36: 0.1u, Capacitor_SMD:C_0603_1608Metric, B.Cu at (272.3, 88.6)
- added C37: 0.1u, Capacitor_SMD:C_0603_1608Metric, F.Cu at (254.8, 91.4)
- added C38: 0.1uF, Capacitor_SMD:C_0603_1608Metric, B.Cu at (173.2, 185.9)
- added C39: 0.1uF, Capacitor_SMD:C_0603_1608Metric, B.Cu at (151.4, 186.9)
- added C4: 0.1uF, Capacitor_SMD:C_0603_1608Metric, F.Cu at (208.9, 130.9)
- added C40: 10u, Capacitor_SMD:C_0805_2012Metric, F.Cu at (284.5, 99.3)
- added C5: 1uF, Capacitor_SMD:C_0603_1608Metric, F.Cu at (208.1, 149.5)
- added C6: 0.01uF, Capacitor_SMD:C_0603_1608Metric, F.Cu at (210.4, 149.5)
- added C7: 0.01uF, Capacitor_SMD:C_0603_1608Metric, F.Cu at (198.4, 136.9)
- added C8: 2.2uF, Capacitor_SMD:C_1206_3216Metric, F.Cu at (205.8, 130.2)
- added C9: 10pF C0G, Capacitor_SMD:C_0603_1608Metric, F.Cu at (222.6, 138.0)
- added D3: LED, ECE445L:LED_D5.0mm, F.Cu at (179.8, 127.8)
- added D4: LED, ECE445L:LED_D5.0mm, F.Cu at (170.7, 127.8)
- added J1: JTAG, ECE445L:PinHeader_1x05_P2.54mm_Vertical, F.Cu at (185.9, 194.3)
- added J2: AudioJack, ECE445L:Jack_3.5mm_CUI_SJ1-3523N_Horizontal, F.Cu at (320.7, 105.2)
- added J3: 2479774-1, ECE445L:24797741, F.Cu at (135.5, 95.0)
- added J4: EK-TM4C123GXL, ECE445L:ti_EKTM4C123GXL, B.Cu at (211.6, 157.7)
- added Q10, Q18: PZT2222A, Package_TO_SOT_SMD:SOT-223-3_TabPin2, F.Cu at (293.2, 88.9)
- added Q11: PZT2222A, Package_TO_SOT_SMD:SOT-223-3_TabPin2, B.Cu at (279.2, 112.3)
- added Q12: PZT2222A, Package_TO_SOT_SMD:SOT-223-3_TabPin2, B.Cu at (278.9, 82.0)
- added Q13: PZT2222A, Package_TO_SOT_SMD:SOT-223-3_TabPin2, B.Cu at (287.3, 112.3)
- added Q14: PZT2222A, Package_TO_SOT_SMD:SOT-223-3_TabPin2, B.Cu at (279.2, 102.6)
- added Q15: PZT2222A, Package_TO_SOT_SMD:SOT-223-3_TabPin2, B.Cu at (287.3, 102.6)
- added Q16: PZT2222A, Package_TO_SOT_SMD:SOT-223-3_TabPin2, B.Cu at (286.3, 82.0)
- added Q17: PZT2222A, Package_TO_SOT_SMD:SOT-223-3_TabPin2, F.Cu at (293.4, 79.7)
- added Q2: PZT2222A, Package_TO_SOT_SMD:SOT-223-3_TabPin2, B.Cu at (192.8, 83.3)
- added Q3: PZT2222A, Package_TO_SOT_SMD:SOT-223-3_TabPin2, B.Cu at (200.9, 93.0)
- added Q4: PZT2222A, Package_TO_SOT_SMD:SOT-223-3_TabPin2, B.Cu at (192.8, 93.0)
- added Q5: PZT2222A, Package_TO_SOT_SMD:SOT-223-3_TabPin2, B.Cu at (193.8, 113.5)
- added Q6: PZT2222A, Package_TO_SOT_SMD:SOT-223-3_TabPin2, B.Cu at (201.2, 113.5)
- added Q7: PZT2222A, Package_TO_SOT_SMD:SOT-223-3_TabPin2, F.Cu at (197.6, 116.0)
- added Q8: PZT2222A, Package_TO_SOT_SMD:SOT-223-3_TabPin2, F.Cu at (186.7, 115.8)
- added Q9: PZT2222A, Package_TO_SOT_SMD:SOT-223-3_TabPin2, F.Cu at (186.8, 106.7)
- added R10: 10k, Resistor_SMD:R_0603_1608Metric, F.Cu at (198.9, 93.5)
- added R11: 20k, Resistor_SMD:R_0603_1608Metric, F.Cu at (200.4, 93.5)
- added R12: 10k, Resistor_SMD:R_0603_1608Metric, F.Cu at (217.4, 105.7)
- added R13: 10k, Resistor_SMD:R_0603_1608Metric, B.Cu at (208.3, 114.3)
- added R14: 10k, Resistor_SMD:R_0603_1608Metric, F.Cu at (203.2, 112.0)
- added R15: 100k, Resistor_SMD:R_0603_1608Metric, F.Cu at (219.2, 114.6)
- added R16: 100k, Resistor_SMD:R_0603_1608Metric, F.Cu at (217.2, 114.6)
- added R17: 20k, Resistor_SMD:R_0603_1608Metric, F.Cu at (203.1, 113.5)
- added R18: 10k, Resistor_SMD:R_0603_1608Metric, F.Cu at (207.0, 105.9)
- added R19: 10k, Resistor_SMD:R_0603_1608Metric, F.Cu at (204.0, 99.5)
- added R2: 10k, Resistor_SMD:R_0603_1608Metric, F.Cu at (215.1, 89.4)
- added R20: 10k, Resistor_SMD:R_0603_1608Metric, F.Cu at (198.6, 83.3)
- added R21: 200k, Resistor_SMD:R_0603_1608Metric, F.Cu at (192.8, 93.5)
- added R22: 200k, Resistor_SMD:R_0603_1608Metric, F.Cu at (194.8, 93.5)
- added R23: 100k, Resistor_SMD:R_0603_1608Metric, F.Cu at (189.7, 100.6)
- added R24: 100k, Resistor_SMD:R_0603_1608Metric, B.Cu at (194.6, 104.6)
- added R25: 100k, Resistor_SMD:R_0603_1608Metric, B.Cu at (194.6, 102.9)
- added R26: 100k, Resistor_SMD:R_0603_1608Metric, F.Cu at (198.6, 110.2)
- added R27: 100k, Resistor_SMD:R_0603_1608Metric, F.Cu at (195.6, 110.2)
- added R28: 100k, Resistor_SMD:R_0603_1608Metric, B.Cu at (188.0, 108.0)
- added R29: 10k, Resistor_SMD:R_0603_1608Metric, F.Cu at (260.9, 106.2)
- added R3: 10k, Resistor_SMD:R_0603_1608Metric, F.Cu at (202.4, 82.0)
- added R30: 10k, Resistor_SMD:R_0603_1608Metric, F.Cu at (264.9, 106.2)
- added R31: 10k, Resistor_SMD:R_0603_1608Metric, F.Cu at (276.9, 108.7)
- added R32: 10k, Resistor_SMD:R_0603_1608Metric, F.Cu at (279.6, 108.0)
- added R33: 20k, Resistor_SMD:R_0603_1608Metric, F.Cu at (279.5, 109.5)
- added R34: 100k, Resistor_SMD:R_0603_1608Metric, F.Cu at (263.2, 99.6)
- added R35: 100k, Resistor_SMD:R_0603_1608Metric, F.Cu at (261.4, 99.6)
- added R36: 10k, Resistor_SMD:R_0603_1608Metric, F.Cu at (277.1, 99.6)
- added R37: 10k, Resistor_SMD:R_0603_1608Metric, F.Cu at (272.0, 91.4)
- added R38: 10k, Resistor_SMD:R_0603_1608Metric, F.Cu at (281.2, 102.1)
- added R39: 20k, Resistor_SMD:R_0603_1608Metric, F.Cu at (279.7, 102.1)
- added R4: 10k, Resistor_SMD:R_0603_1608Metric, F.Cu at (203.2, 86.9)
- added R40: 10k, Resistor_SMD:R_0603_1608Metric, F.Cu at (262.7, 89.9)
- added R41: 10k, Resistor_SMD:R_0603_1608Metric, B.Cu at (271.7, 81.3)
- added R42: 10k, Resistor_SMD:R_0603_1608Metric, F.Cu at (276.9, 83.6)
- added R43: 100k, Resistor_SMD:R_0603_1608Metric, F.Cu at (260.9, 81.0)
- added R44: 100k, Resistor_SMD:R_0603_1608Metric, F.Cu at (262.9, 81.0)
- added R45: 20k, Resistor_SMD:R_0603_1608Metric, F.Cu at (276.9, 82.0)
- added R46: 10k, Resistor_SMD:R_0603_1608Metric, F.Cu at (273.0, 89.7)
- added R47: 10k, Resistor_SMD:R_0603_1608Metric, F.Cu at (276.1, 96.1)
- added R48: 10k, Resistor_SMD:R_0603_1608Metric, F.Cu at (281.4, 112.3)
- added R49: 200k, Resistor_SMD:R_0603_1608Metric, F.Cu at (287.3, 100.1)
- added R5: 20k, Resistor_SMD:R_0603_1608Metric, F.Cu at (202.4, 84.1)
- added R50: 200k, Resistor_SMD:R_0603_1608Metric, F.Cu at (289.3, 100.1)
- added R51: 100k, Resistor_SMD:R_0603_1608Metric, F.Cu at (289.1, 95.5)
- added R52: 100k, Resistor_SMD:R_0603_1608Metric, B.Cu at (285.4, 91.2)
- added R53: 100k, Resistor_SMD:R_0603_1608Metric, B.Cu at (285.5, 93.0)
- added R54: 100k, Resistor_SMD:R_0603_1608Metric, F.Cu at (285.0, 82.5)
- added R55: 100k, Resistor_SMD:R_0603_1608Metric, F.Cu at (285.0, 80.8)
- added R56: 100k, Resistor_SMD:R_0603_1608Metric, F.Cu at (287.0, 85.6)
- added R57: 75K, Resistor_SMD:R_0603_1608Metric, F.Cu at (287.8, 83.3)
- added R58: 50, Resistor_SMD:R_0603_1608Metric, F.Cu at (310.6, 100.1)
- added R59: 50, Resistor_SMD:R_0603_1608Metric, F.Cu at (310.4, 110.2)
- added R6: 100k, Resistor_SMD:R_0603_1608Metric, F.Cu at (216.9, 96.0)
- added R60: 1k, Resistor_SMD:R_0603_1608Metric, B.Cu at (236.7, 120.1)
- added R61: 47k, Resistor_SMD:R_0603_1608Metric, B.Cu at (240.5, 120.1)
- added R62: 10k, Resistor_SMD:R_0603_1608Metric, B.Cu at (238.8, 115.1)
- added R63: 10k, Resistor_SMD:R_0603_1608Metric, B.Cu at (284.5, 190.5)
- added R64: 1M, Resistor_SMD:R_0603_1608Metric, F.Cu at (212.9, 148.8)
- added R65: 10k, Resistor_SMD:R_0603_1608Metric, B.Cu at (246.1, 190.5)
- added R66: 10k, Resistor_SMD:R_0603_1608Metric, B.Cu at (265.4, 190.5)
- added R67: 10k, Resistor_SMD:R_0603_1608Metric, B.Cu at (246.4, 175.3)
- added R68: 10k, Resistor_SMD:R_0603_1608Metric, B.Cu at (265.4, 175.2)
- added R69: 10k, Resistor_SMD:R_0603_1608Metric, B.Cu at (303.3, 190.5)
- added R7: 100k, Resistor_SMD:R_0603_1608Metric, F.Cu at (218.7, 96.0)
- added R70: 10k, ECE445L:P120PK-Y25BR10K, F.Cu at (252.5, 158.8)
- added R71: 10k, ECE445L:P120PK-Y25BR10K, F.Cu at (309.6, 158.8)
- added R72: 10k, ECE445L:P120PK-Y25BR10K, F.Cu at (271.5, 158.8)
- added R73: 10k, ECE445L:P120PK-Y25BR10K, F.Cu at (309.9, 136.9)
- added R74: 10k, ECE445L:P120PK-Y25BR10K, F.Cu at (290.6, 136.0)
- added R75: 10k, ECE445L:P120PK-Y25BR10K, F.Cu at (271.5, 136.0)
- added R76: 10k, ECE445L:P120PK-Y25BR10K, F.Cu at (252.5, 136.0)
- added R77: 0, Resistor_SMD:R_0603_1608Metric, F.Cu at (193.8, 78.7)
- added R78: 2k, Resistor_SMD:R_0603_1608Metric, B.Cu at (182.4, 131.1)
- added R79: 2k, Resistor_SMD:R_0603_1608Metric, B.Cu at (173.2, 131.4)
- added R8: 10k, Resistor_SMD:R_0603_1608Metric, F.Cu at (202.9, 96.0)
- added R80: 10k, ECE445L:P120PK-Y25BR10K, F.Cu at (290.6, 158.8)
- added R81: 10k, Resistor_SMD:R_0603_1608Metric, B.Cu at (284.5, 175.3)
- added R82: 75K, Resistor_SMD:R_0603_1608Metric, B.Cu at (188.0, 111.8)
- added R83: 0, Resistor_SMD:R_0603_1608Metric, F.Cu at (198.6, 79.2)
- added R84: 10k, Resistor_SMD:R_0603_1608Metric, B.Cu at (303.5, 175.3)
- added R85: 5K1, Resistor_SMD:R_0603_1608Metric, F.Cu at (142.1, 96.0)
- added R86: 5K1, Resistor_SMD:R_0603_1608Metric, F.Cu at (142.1, 94.0)
- added R9: 10k, Resistor_SMD:R_0603_1608Metric, F.Cu at (199.6, 96.0)
- added SW6: Delay, ECE445L:SW_PUSH_6mm, F.Cu at (287.3, 171.5)
- added SW7: Tempo, ECE445L:SW_PUSH_6mm, F.Cu at (306.4, 171.5)
- added SW8: Reset, Button_Switch_THT:SW_PUSH_6mm, F.Cu at (287.3, 186.8)
- added SW9: SW_SPST, ECE445L:SW-T3-1A-A-A3-S1, F.Cu at (161.8, 91.4)
- added TP1: +VRail, ECE445L:Testpoint_1x02_P2.54mm, F.Cu at (149.3, 83.1)
- added TP10: L_Treble, ECE445L:Testpoint_1x02_P2.54mm, F.Cu at (250.5, 85.1)
- added TP11: L_Buff, ECE445L:Testpoint_1x02_P2.54mm, F.Cu at (294.1, 109.0)
- added TP12: L_Out, ECE445L:Testpoint_1x02_P2.54mm, F.Cu at (294.4, 97.8)
- added TP13: +VRef, ECE445L:Testpoint_1x02_P2.54mm, F.Cu at (241.0, 79.0)
- added TP2: 3V3, ECE445L:Testpoint_1x02_P2.54mm, F.Cu at (174.5, 80.8)
- added TP3: R_Bass, ECE445L:Testpoint_1x02_P2.54mm, F.Cu at (228.6, 82.8)
- added TP4: R_Mid, ECE445L:Testpoint_1x02_P2.54mm, F.Cu at (229.1, 89.4)
- added TP5: R_Treble, ECE445L:Testpoint_1x02_P2.54mm, F.Cu at (229.6, 110.5)
- added TP6: R_Buff, ECE445L:Testpoint_1x02_P2.54mm, F.Cu at (185.9, 86.6)
- added TP7: R_Out, ECE445L:Testpoint_1x02_P2.54mm, F.Cu at (185.7, 97.8)
- added TP8: L_Bass, ECE445L:Testpoint_1x02_P2.54mm, F.Cu at (251.5, 112.8)
- added TP9: L_Mid, ECE445L:Testpoint_1x02_P2.54mm, F.Cu at (251.0, 106.2)
- added U10: OPA2350, ECE445L:DIP-8_W7.62mm_LongPads, F.Cu at (206.8, 116.8)
- added U11: OPA2350, ECE445L:DIP-8_W7.62mm_LongPads, F.Cu at (273.3, 109.2)
- added U12: OPA2350, ECE445L:DIP-8_W7.62mm_LongPads, F.Cu at (273.3, 94.0)
- added U13: OPA2350, ECE445L:DIP-8_W7.62mm_LongPads, F.Cu at (278.7, 96.0)
- added U14: OPA2350, ECE445L:DIP-8_W7.62mm_LongPads, F.Cu at (201.4, 99.6)
- added U15: TLV5616, ECE445L:DIP-8_W7.62mm_LongPads, F.Cu at (247.9, 94.0)
- added U16: Adafruit ST7735R, ECE445L:adafruit_st7735r2, F.Cu at (161.8, 164.1)
- added U4: LM2937ET-3.3_NOPB, ECE445L:TO254P470X1028X1955-3P, B.Cu at (159.8, 83.2)
- added U5: TLV5616, ECE445L:DIP-8_W7.62mm_LongPads, F.Cu at (232.2, 101.6)
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Connections:
- C1 pad 1: unconnected-(C1-Pad1) -> +3V3
- C1 pad 2: unconnected-(C1-Pad2) -> GND
- C2 pad 1: unconnected-(C2-Pad1) -> /Lab7_microcontroller/LDO
- C2 pad 2: unconnected-(C2-Pad2) -> GND
- Q1 pad 1: unconnected-(Q1-D-Pad1) -> PB2
- Q1 pad 2: unconnected-(Q1-D-Pad2) -> Net-(Q1-C)
- Q1 pad 3: unconnected-(Q1-G-Pad3) -> GND
- R1 pad 1: unconnected-(R1-Pad1) -> Net-(C15-Pad2)
- R1 pad 2: unconnected-(R1-Pad2) -> Vin_R
- SW1 pad 2: /Lab7_Input/SW_UP -> PB0
- SW2 pad 2: /Lab7_Input/SW_DOWN -> PB1
- SW3 pad 2: /Lab7_Input/SW_LEFT -> PB2
- SW4 pad 2: /Lab7_Input/SW_RIGHT -> PB3
- SW5 pad 2: /Lab7_Input/SW_MODE -> PB4
- U2 pad 1: GND -> unconnected-(U2-GPIO36-Pad1)
- U2 pad 10: unconnected-(U2-LITE-Pad10) -> LAUDIO_FS
- U2 pad 7: unconnected-(U2-MOSI-Pad7) -> RAUDIO_OUT
- U2 pad 8: unconnected-(U2-SCK-Pad8) -> RAUDIO_CLK
- U2 pad 9: unconnected-(U2-MISO-Pad9) -> RAUDIO_FS
- U3 pad 1: unconnected-(U3-RxD-Pad1) -> ESP_IN_USB_OUT
- U3 pad 2: unconnected-(U3-GPIO0-Pad2) -> ESP_OUT_USB_IN
- U3 pad 4: unconnected-(U3-GND-Pad4) -> (no net)
Routing:
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Other:
- board size 115 x 94 mm -> 192.5 x 127 mm

Commit message: Pushing layout for merge
Parts:
- moved H4 1.30 mm to (319.0, 195.1)
- moved H1 1.05 mm to (136.7, 195.1)
- moved H2 0.51 mm to (136.7, 78.2)
- moved H3 0.36 mm to (319.0, 78.2)
Changed lines of the file:
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@@
 	(footprint "ECE445L:MountingHole_4_40"
 		(layer "F.Cu")
-		(at 320.294 194.818)
+		(at 319.024 195.072)
 		(descr "Mounting Hole 0.125in")
 		(tags "mounting hole 0.125in 4_40")
@@
 	(footprint "ECE445L:MountingHole_4_40"
 		(layer "F.Cu")
-		(at 136.652 77.724)
+		(at 136.652 78.232)
 		(descr "Mounting Hole 0.125in")
 		(tags "mounting hole 0.125in 4_40")
@@
 	(footprint "ECE445L:MountingHole_4_40"
 		(layer "F.Cu")
-		(at 135.636 195.326)
+		(at 136.652 195.072)
 		(descr "Mounting Hole 0.125in")
 		(tags "mounting hole 0.125in 4_40")
@@
 	(footprint "ECE445L:MountingHole_4_40"
 		(layer "F.Cu")
-		(at 319.278 78.486)
+		(at 319.024 78.232)
 		(descr "Mounting Hole 0.125in")
 		(tags "mounting hole 0.125in 4_40")
@@
 			(layer "B.SilkS")
 		)
-		(fp_circle
-			(center 12.43 23.86)
-			(end 12.43 22.36)
-			(stroke
-				(width 0.1)
-				(type default)
-			)
-			(fill no)
-			(layer "Edge.Cuts")
-		)
-		(fp_circle
-			(center 12.43 -22.14)
-			(end 12.43 -23.64)
-			(stroke
-				(width 0.1)
-				(type default)
-			)
-			(fill no)
-			(layer "Edge.Cuts")
-		)
-		(fp_circle
-			(center -10.57 23.86)
-			(end -10.57 22.36)
-			(stroke
-				(width 0.1)
-				(type default)
-			)
-			(fill no)
-			(layer "Edge.Cuts")
-		)
-		(fp_circle
-			(center -10.57 -22.14)
-			(end -10.57 -23.64)
-			(stroke
-				(width 0.1)
-				(type default)
-			)
-			(fill no)
-			(layer "Edge.Cuts")
-		)
 		(fp_text user "GPIO13"

Commit message: Parts layout part 2
Parts:
- moved C39 368.3 mm to (519.7, 191.3)
- moved SW6 260.6 mm to (34.3, 109.3)
- moved SW7 260.6 mm to (53.3, 109.3)
- moved R84 260.4 mm to (51.0, 111.5)
- moved R81 260.4 mm to (32.0, 111.8)
- moved R71 259.7 mm to (56.6, 100.4)
- moved R80 259.7 mm to (37.6, 100.4)
- moved SW5 254.1 mm to (70.2, 93.3)
- moved R69 253.5 mm to (67.6, 97.3), turned to -90 degrees
- moved R67 236.7 mm to (32.0, 74.9)
- moved R68 236.7 mm to (51.0, 74.9)
- moved SW3 236.7 mm to (34.3, 72.5)
- moved SW4 236.7 mm to (53.3, 72.5)
- moved R70 235.1 mm to (37.6, 63.6)
- moved R72 235.1 mm to (56.6, 63.6)
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Routing:
- net /Lab7_microcontroller/OSC2: track 3.55 -> 0.00 mm
- net /Lab7_microcontroller/OSC1: track 3.55 -> 0.00 mm
Other:
- board size 192.5 x 127 mm -> 152.4 x 127 mm
- board text added: "Bass"
- board text added: "Delay"
- board text added: "Distortion"
- board text added: "Flanger"
- board text added: "Mid"
- board text added: "Space for Both Audio Channels"
- board text added: "Tempo"
- board text added: "Treble"
- board text added: "USB -> UART Converter"
- board text added: "Volume"

Commit message: Rough draft layout - need to remove tm4c chip
Parts:
- removed the R63 at (123.5, 96.5)
- removed the R83 at (236.7, 57.4)
- removed the SW8 at (126.3, 93.8)
- removed TP10: L_Treble, ECE445L:Testpoint_1x02_P2.54mm
- removed TP11: L_Buff, ECE445L:Testpoint_1x02_P2.54mm
- removed the TP13 at (279.1, 57.1)
- removed the TP4 at (267.2, 67.6)
- removed TP5: R_Treble, ECE445L:Testpoint_1x02_P2.54mm
- removed TP6: R_Buff, ECE445L:Testpoint_1x02_P2.54mm
- removed TP7: R_Out, ECE445L:Testpoint_1x02_P2.54mm
- removed TP8: L_Bass, ECE445L:Testpoint_1x02_P2.54mm
- removed TP9: L_Mid, ECE445L:Testpoint_1x02_P2.54mm
- added D3: 1N914, ECE445L:Testpoint_1x02_P2.54mm, B.Cu at (163.3, 89.7)
- added D4: 1N914, ECE445L:Testpoint_1x02_P2.54mm, B.Cu at (163.3, 94.0)
- added R28: 40k, Resistor_SMD:R_0603_1608Metric_Pad0.98x0.95mm_HandSolder, F.Cu at (117.4, 69.6)
- added R29: 3.3k, Resistor_SMD:R_0603_1608Metric_Pad0.98x0.95mm_HandSolder, F.Cu at (118.4, 66.5)
- added R59: 40k, Resistor_SMD:R_0603_1608Metric_Pad0.98x0.95mm_HandSolder, B.Cu at (163.3, 66.2)
- added R60: 3.3k, Resistor_SMD:R_0603_1608Metric_Pad0.98x0.95mm_HandSolder, B.Cu at (166.8, 61.6)
- added TP3: +VRef, ECE445L:Testpoint_1x02_P2.54mm, F.Cu at (160.8, 29.2)
- C1: renamed from C12; footprint Capacitor_SMD:C_0603_1608Metric -> Capacitor_SMD:C_0603_1608Metric_Pad1.08x0.95mm_HandSolder
- C10: renamed from C4; footprint Capacitor_SMD:C_0603_1608Metric -> Capacitor_SMD:C_0603_1608Metric_Pad1.08x0.95mm_HandSolder
- C11: renamed from C6; footprint Capacitor_SMD:C_0603_1608Metric -> Capacitor_SMD:C_0603_1608Metric_Pad1.08x0.95mm_HandSolder
- C12: renamed from C9; footprint Capacitor_SMD:C_0603_1608Metric -> Capacitor_SMD:C_0603_1608Metric_Pad1.08x0.95mm_HandSolder
- C13: renamed from C10; footprint Capacitor_SMD:C_0603_1608Metric -> Capacitor_SMD:C_0603_1608Metric_Pad1.08x0.95mm_HandSolder
- C14: renamed from C11; footprint Capacitor_SMD:C_0603_1608Metric -> Capacitor_SMD:C_0603_1608Metric_Pad1.08x0.95mm_HandSolder
- C15: renamed from C19; footprint Capacitor_SMD:C_0603_1608Metric -> Capacitor_SMD:C_0603_1608Metric_Pad1.08x0.95mm_HandSolder; moved to B.Cu
- C16: renamed from C15; value 27n -> 30n; footprint Capacitor_SMD:C_0603_1608Metric -> Capacitor_SMD:C_0603_1608Metric_Pad1.08x0.95mm_HandSolder
- C17: renamed from C20; footprint Capacitor_SMD:C_0603_1608Metric -> Capacitor_SMD:C_0603_1608Metric_Pad1.08x0.95mm_HandSolder; moved to B.Cu
- C18: renamed from C16; value 27n -> 30n; footprint Capacitor_SMD:C_0603_1608Metric -> Capacitor_SMD:C_0603_1608Metric_Pad1.08x0.95mm_HandSolder; moved to F.Cu
- C19: renamed from C17; value 10n -> 9.5n; footprint Capacitor_SMD:C_0603_1608Metric -> Capacitor_SMD:C_0603_1608Metric_Pad1.08x0.95mm_HandSolder
- C2: renamed from C13; footprint Capacitor_SMD:C_0805_2012Metric -> Capacitor_SMD:C_0805_2012Metric_Pad1.18x1.45mm_HandSolder; moved to F.Cu
- C20: renamed from C18; value 3.5n -> 3.7n; footprint Capacitor_SMD:C_0603_1608Metric -> Capacitor_SMD:C_0603_1608Metric_Pad1.08x0.95mm_HandSolder; moved to B.Cu
- C21: renamed from C22; footprint Capacitor_SMD:C_0603_1608Metric -> Capacitor_SMD:C_0603_1608Metric_Pad1.08x0.95mm_HandSolder
- C22: renamed from C23; footprint Capacitor_SMD:C_0603_1608Metric -> Capacitor_SMD:C_0603_1608Metric_Pad1.08x0.95mm_HandSolder; moved to F.Cu
- C23: renamed from C24; footprint Capacitor_SMD:C_0603_1608Metric -> Capacitor_SMD:C_0603_1608Metric_Pad1.08x0.95mm_HandSolder
- C24: renamed from C25; footprint Capacitor_SMD:C_0603_1608Metric -> Capacitor_SMD:C_0603_1608Metric_Pad1.08x0.95mm_HandSolder; moved to F.Cu
- C25: renamed from C21; footprint Capacitor_SMD:C_0805_2012Metric -> Capacitor_SMD:C_0805_2012Metric_Pad1.18x1.45mm_HandSolder; moved to B.Cu
- C26: footprint Capacitor_SMD:C_0603_1608Metric -> Capacitor_SMD:C_0603_1608Metric_Pad1.08x0.95mm_HandSolder; moved to B.Cu
- C27: renamed from C31; footprint Capacitor_SMD:C_0603_1608Metric -> Capacitor_SMD:C_0603_1608Metric_Pad1.08x0.95mm_HandSolder
- C28: renamed from C27; value 27n -> 30n; footprint Capacitor_SMD:C_0603_1608Metric -> Capacitor_SMD:C_0603_1608Metric_Pad1.08x0.95mm_HandSolder
- C29: renamed from C32; footprint Capacitor_SMD:C_0603_1608Metric -> Capacitor_SMD:C_0603_1608Metric_Pad1.08x0.95mm_HandSolder
- C3: renamed from C14; footprint Capacitor_SMD:C_0603_1608Metric -> Capacitor_SMD:C_0603_1608Metric_Pad1.08x0.95mm_HandSolder
- C30: renamed from C28; value 27n -> 30n; footprint Capacitor_SMD:C_0603_1608Metric -> Capacitor_SMD:C_0603_1608Metric_Pad1.08x0.95mm_HandSolder
- C31: renamed from C29; value 10n -> 9.5n; footprint Capacitor_SMD:C_0603_1608Metric -> Capacitor_SMD:C_0603_1608Metric_Pad1.08x0.95mm_HandSolder
- C32: renamed from C30; value 3.5n -> 3.7n; footprint Capacitor_SMD:C_0603_1608Metric -> Capacitor_SMD:C_0603_1608Metric_Pad1.08x0.95mm_HandSolder; moved to B.Cu
- C33, C35, C36: footprint Capacitor_SMD:C_0603_1608Metric -> Capacitor_SMD:C_0603_1608Metric_Pad1.08x0.95mm_HandSolder
- C34: footprint Capacitor_SMD:C_0603_1608Metric -> Capacitor_SMD:C_0603_1608Metric_Pad1.08x0.95mm_HandSolder; moved to F.Cu
- C37: renamed from C40; footprint Capacitor_SMD:C_0805_2012Metric -> Capacitor_SMD:C_0805_2012Metric_Pad1.18x1.45mm_HandSolder; moved to B.Cu
- C38: renamed from C37; footprint Capacitor_SMD:C_0603_1608Metric -> Capacitor_SMD:C_0603_1608Metric_Pad1.08x0.95mm_HandSolder
- C39: renamed from C38; footprint Capacitor_SMD:C_0603_1608Metric -> Capacitor_SMD:C_0603_1608Metric_Pad1.08x0.95mm_HandSolder; moved to F.Cu
- C4: renamed from C7; footprint Capacitor_SMD:C_0603_1608Metric -> Capacitor_SMD:C_0603_1608Metric_Pad1.08x0.95mm_HandSolder
- C40: renamed from C39; footprint Capacitor_SMD:C_0603_1608Metric -> Capacitor_SMD:C_0603_1608Metric_Pad1.08x0.95mm_HandSolder; moved to F.Cu
- C5: renamed from C1; footprint Capacitor_SMD:C_0603_1608Metric -> Capacitor_SMD:C_0603_1608Metric_Pad1.08x0.95mm_HandSolder
- C6: renamed from C5; footprint Capacitor_SMD:C_0603_1608Metric -> Capacitor_SMD:C_0603_1608Metric_Pad1.08x0.95mm_HandSolder
- C7: renamed from C8; footprint Capacitor_SMD:C_1206_3216Metric -> Capacitor_SMD:C_1206_3216Metric_Pad1.33x1.80mm_HandSolder
- C8: renamed from C3; footprint Capacitor_SMD:C_0603_1608Metric -> Capacitor_SMD:C_0603_1608Metric_Pad1.08x0.95mm_HandSolder
- C9: renamed from C2; footprint Capacitor_SMD:C_0603_1608Metric -> Capacitor_SMD:C_0603_1608Metric_Pad1.08x0.95mm_HandSolder
- J3: renamed from J1; moved to B.Cu
- Q13, Q15: moved to F.Cu
- Q17, Q18, Q7, Q8, Q9: moved to B.Cu
- Q3: renamed from Q6; moved to F.Cu
- Q4: renamed from Q2; moved to F.Cu
- R1: renamed from R86; footprint Resistor_SMD:R_0603_1608Metric -> Resistor_SMD:R_0603_1608Metric_Pad0.98x0.95mm_HandSolder
- R10: renamed from R15; footprint Resistor_SMD:R_0603_1608Metric -> Resistor_SMD:R_0603_1608Metric_Pad0.98x0.95mm_HandSolder; moved to B.Cu
- R11: renamed from R16; footprint Resistor_SMD:R_0603_1608Metric -> Resistor_SMD:R_0603_1608Metric_Pad0.98x0.95mm_HandSolder; moved to B.Cu
- R12: renamed from R17; footprint Resistor_SMD:R_0603_1608Metric -> Resistor_SMD:R_0603_1608Metric_Pad0.98x0.95mm_HandSolder; moved to B.Cu
- R13: renamed from R5; footprint Resistor_SMD:R_0603_1608Metric -> Resistor_SMD:R_0603_1608Metric_Pad0.98x0.95mm_HandSolder; moved to B.Cu
- R14: footprint Resistor_SMD:R_0603_1608Metric -> Resistor_SMD:R_0603_1608Metric_Pad0.98x0.95mm_HandSolder; moved to B.Cu
- R15: renamed from R3; footprint Resistor_SMD:R_0603_1608Metric -> Resistor_SMD:R_0603_1608Metric_Pad0.98x0.95mm_HandSolder
- R16: renamed from R13; footprint Resistor_SMD:R_0603_1608Metric -> Resistor_SMD:R_0603_1608Metric_Pad0.98x0.95mm_HandSolder
- R17: renamed from R4; footprint Resistor_SMD:R_0603_1608Metric -> Resistor_SMD:R_0603_1608Metric_Pad0.98x0.95mm_HandSolder; moved to B.Cu
- R18: renamed from R6; footprint Resistor_SMD:R_0603_1608Metric -> Resistor_SMD:R_0603_1608Metric_Pad0.98x0.95mm_HandSolder
- R19: renamed from R7; footprint Resistor_SMD:R_0603_1608Metric -> Resistor_SMD:R_0603_1608Metric_Pad0.98x0.95mm_HandSolder
- R2: renamed from R85; footprint Resistor_SMD:R_0603_1608Metric -> Resistor_SMD:R_0603_1608Metric_Pad0.98x0.95mm_HandSolder
- R20: renamed from R11; footprint Resistor_SMD:R_0603_1608Metric -> Resistor_SMD:R_0603_1608Metric_Pad0.98x0.95mm_HandSolder
- R21: renamed from R10; footprint Resistor_SMD:R_0603_1608Metric -> Resistor_SMD:R_0603_1608Metric_Pad0.98x0.95mm_HandSolder
- R22: renamed from R9; footprint Resistor_SMD:R_0603_1608Metric -> Resistor_SMD:R_0603_1608Metric_Pad0.98x0.95mm_HandSolder
- R23: renamed from R77; footprint Resistor_SMD:R_0603_1608Metric -> Resistor_SMD:R_0603_1608Metric_Pad0.98x0.95mm_HandSolder
- R24: renamed from R8; footprint Resistor_SMD:R_0603_1608Metric -> Resistor_SMD:R_0603_1608Metric_Pad0.98x0.95mm_HandSolder; moved to B.Cu
- R25: renamed from R19; value 10k -> 7.5k; footprint Resistor_SMD:R_0603_1608Metric -> Resistor_SMD:R_0603_1608Metric_Pad0.98x0.95mm_HandSolder
- R26: renamed from R20; footprint Resistor_SMD:R_0603_1608Metric -> Resistor_SMD:R_0603_1608Metric_Pad0.98x0.95mm_HandSolder
- R27: renamed from R18; footprint Resistor_SMD:R_0603_1608Metric -> Resistor_SMD:R_0603_1608Metric_Pad0.98x0.95mm_HandSolder
- R3: renamed from R60; footprint Resistor_SMD:R_0603_1608Metric -> Resistor_SMD:R_0603_1608Metric_Pad0.98x0.95mm_HandSolder; moved to F.Cu
- R30: renamed from R21; footprint Resistor_SMD:R_0603_1608Metric -> Resistor_SMD:R_0603_1608Metric_Pad0.98x0.95mm_HandSolder; moved to B.Cu
- R31: renamed from R22; footprint Resistor_SMD:R_0603_1608Metric -> Resistor_SMD:R_0603_1608Metric_Pad0.98x0.95mm_HandSolder; moved to B.Cu
- R32: renamed from R24; footprint Resistor_SMD:R_0603_1608Metric -> Resistor_SMD:R_0603_1608Metric_Pad0.98x0.95mm_HandSolder
- R33: renamed from R23; footprint Resistor_SMD:R_0603_1608Metric -> Resistor_SMD:R_0603_1608Metric_Pad0.98x0.95mm_HandSolder; moved to B.Cu
- R34: renamed from R25; footprint Resistor_SMD:R_0603_1608Metric -> Resistor_SMD:R_0603_1608Metric_Pad0.98x0.95mm_HandSolder
- R35: renamed from R26; footprint Resistor_SMD:R_0603_1608Metric -> Resistor_SMD:R_0603_1608Metric_Pad0.98x0.95mm_HandSolder
- R36: renamed from R27; footprint Resistor_SMD:R_0603_1608Metric -> Resistor_SMD:R_0603_1608Metric_Pad0.98x0.95mm_HandSolder
- R37: renamed from R82; footprint Resistor_SMD:R_0603_1608Metric -> Resistor_SMD:R_0603_1608Metric_Pad0.98x0.95mm_HandSolder; moved to F.Cu
- R38: renamed from R28; footprint Resistor_SMD:R_0603_1608Metric -> Resistor_SMD:R_0603_1608Metric_Pad0.98x0.95mm_HandSolder; moved to F.Cu
- R39: renamed from R29; footprint Resistor_SMD:R_0603_1608Metric -> Resistor_SMD:R_0603_1608Metric_Pad0.98x0.95mm_HandSolder; moved to B.Cu
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- renumbered D3 to D1, D4 to D2, J3 to J1, J4 to J2, J2 to J4, Q5 to Q1, Q1 to Q2, Q3 to Q5, Q4 to Q6, R70 to R77, R72 to R78, R80 to R79, R71 to R80, R73 to R81, R74 to R82, R75 to R83, R76 to R84, SW9 to SW1, SW1 to SW2, SW2 to SW3, SW3 to SW4, SW4 to SW5, SW5 to SW6, SW6 to SW7, SW7 to SW8, TP2 to TP1, TP1 to TP2, TP3 to TP4, U4 to U1, U5 to U10, U6 to U11, U11 to U12, U12 to U13, U13 to U14, U2 to U3, U3 to U4, U1 to U5, U10 to U6, U8 to U7, U9 to U8, U14 to U9
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Connections:
- C19 pad 2: Net-(U9A-+) -> Net-(U8A-+)
- C27 pad 1: Vin -> Vin_L
- C28 pad 2: Net-(C27-Pad2) (its old number) -> Net-(C28-Pad2)
- C31 pad 1: Vin -> Vin_L
- C31 pad 2: Net-(U12A-+) (its old number) -> Net-(U13A-+)
- R18 pad 1: Net-(R6-Pad1) -> Net-(U8A-+)
- R19 pad 2: Net-(R6-Pad1) -> Net-(U8A-+)
- R25 pad 2: Net-(U14A-+) (its old number) -> Net-(U9A-+)
- R26 pad 2: Net-(U14A-+) (its old number) -> Net-(U9A-+)
- R27 pad 1: R_Treble -> Net-(U9A-+)
- R27 pad 2: Net-(U14A-+) (its old number) -> R_Treble
- R39 pad 1: Net-(C27-Pad2) (its old number) -> Vin_L
- R39 pad 2: Vin_L -> Net-(C28-Pad2)
- R41 pad 1: Net-(C27-Pad2) (its old number) -> Net-(C28-Pad2)
- R50 pad 1: Net-(R34-Pad1) -> Net-(U13A-+)
- R51 pad 2: Net-(R34-Pad1) -> Net-(U13A-+)
- R56 pad 1: R_Mid -> L_Mid
- R57 pad 1: R_Bass -> L_Bass
- R58 pad 1: R_Treble -> L_Treble
- R63 pad 1: Net-(U13B-+) (its old number) -> Net-(U14B-+)
- R65 pad 1: GND -> Net-(U14B-+)
- R65 pad 2: Net-(U13B-+) (its old number) -> GND
- R70 pad 2: PB0 -> PF0
- R71 pad 2: PB1 -> PF1
- R72 pad 2: PB2 -> PF2
- R73 pad 2: PB3 -> PF3
- R74 pad 2: PB4 -> PF4
- R79 pad 2: PD1 -> PE4
- R85 pad 1: PB3 -> PD6
- R88 pad 1: PB3 -> PD7
- SW2 pad 2: PB0 -> PF0
- SW3 pad 2: PB1 -> PF1
- SW4 pad 2: PB2 -> PF2
- SW5 pad 2: PB3 -> PF3
- SW6 pad 2: PB4 -> PF4
- U13 pad 3: Net-(U12A-+) (its old number) -> Net-(U13A-+)
- U14 pad 2: L_Buff -> Net-(U14A--)
- U14 pad 5: Net-(U13B-+) (its old number) -> Net-(U14B-+)
- U3 pad 1: unconnected-(U2-GPIO36-Pad1) -> +3V3
- U3 pad 10: LAUDIO_FS -> RAUDIO_FS
- U3 pad 11: LAUDIO_OUT -> LAUDIO_FS
- U3 pad 12: LAUDIO_CLK -> LAUDIO_OUT
- U3 pad 13: GND -> LAUDIO_CLK
- U3 pad 14: +VRail -> GND
- U3 pad 15: unconnected-(U2-GPIO23-Pad15) -> +VRail
- U3 pad 17: TM4C_IN_ESP_OUT -> unconnected-(U3-GPIO22-Pad17)
- U3 pad 18: TM4C_OUT_ESP_IN -> PB0
- U3 pad 19: unconnected-(U2-GPIO21-Pad19) -> PB1
- U3 pad 23: ESP_IN_USB_OUT -> unconnected-(U3-GPIO5-Pad23)
- U3 pad 24: ESP_OUT_USB_IN -> ESP_IN_USB_OUT
- U3 pad 25: unconnected-(U2-GPIO4-Pad25) -> ESP_OUT_USB_IN
- U3 pad 28: GND -> unconnected-(U3-GPIO15-Pad28)
- U3 pad 29: unconnected-(U2-3V3-Pad29) -> GND
- U3 pad 30: (no net) -> unconnected-(U3-3V3-Pad30)
- U3 pad 7: RAUDIO_OUT -> unconnected-(U3-GPIO33-Pad7)
- U3 pad 8: RAUDIO_CLK -> RAUDIO_OUT
- U3 pad 9: RAUDIO_FS -> RAUDIO_CLK
- U4 pad 4: (no net) -> GND
- U5 pad 17: TM4C_IN_ESP_OUT -> PA0
- U5 pad 18: TM4C_OUT_ESP_IN -> PA1
- U5 pad 38: /Lab7_microcontroller/Reset -> +3V3
- U8 pad 3: Net-(U9A-+) -> Net-(U8A-+)
- U9 pad 2: R_Buff -> Net-(U9A--)
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Routing:
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Other:
- board text added: "ECE445L - Lab 7 Nathan DeLaRosa Ashton Knecht Niranjan Telkikar Thompson Troung TA : Michael Chung"
- board text added: "x"
- board text removed: "Space for Both Audio Channels"

Commit message: PCB Layout
Parts:
- removed C11: 0.01uF, Capacitor_SMD:C_0603_1608Metric_Pad1.08x0.95mm_HandSolder
- removed C12, C13: 10pF C0G, Capacitor_SMD:C_0603_1608Metric_Pad1.08x0.95mm_HandSolder
- removed C14: 1uF, Capacitor_SMD:C_0603_1608Metric_Pad1.08x0.95mm_HandSolder
- removed J3: JTAG, ECE445L:PinHeader_1x05_P2.54mm_Vertical
- removed TP13: L_Out, ECE445L:Testpoint_1x02_P2.54mm
- removed U4: FT2322R, Connector_PinHeader_1.00mm:PinHeader_1x04_P1.00mm_Vertical
- removed Y1: ABM3-16.000MHZ-B2-T, ECE445L:ABM3
- added R100: 2k, Resistor_SMD:R_0603_1608Metric_Pad0.98x0.95mm_HandSolder, F.Cu at (100.8, 77.0)
- added R101: 2k, Resistor_SMD:R_0603_1608Metric_Pad0.98x0.95mm_HandSolder, B.Cu at (100.8, 62.7)
- added R102: 2k, Resistor_SMD:R_0603_1608Metric_Pad0.98x0.95mm_HandSolder, B.Cu at (137.9, 75.7)
- added R103: 2k, Resistor_SMD:R_0603_1608Metric_Pad0.98x0.95mm_HandSolder, B.Cu at (133.9, 78.7)
- added R104: 2k, Resistor_SMD:R_0603_1608Metric_Pad0.98x0.95mm_HandSolder, F.Cu at (139.4, 70.1)
- added R105: 2k, Resistor_SMD:R_0603_1608Metric_Pad0.98x0.95mm_HandSolder, B.Cu at (153.9, 62.7)
- added R106: 2k, Resistor_SMD:R_0603_1608Metric_Pad0.98x0.95mm_HandSolder, B.Cu at (147.6, 59.7)
- added R107: 2k, Resistor_SMD:R_0603_1608Metric_Pad0.98x0.95mm_HandSolder, B.Cu at (132.1, 48.8)
- added R108: 2k, Resistor_SMD:R_0603_1608Metric_Pad0.98x0.95mm_HandSolder, B.Cu at (137.9, 49.1)
- added R109: 2k, Resistor_SMD:R_0603_1608Metric_Pad0.98x0.95mm_HandSolder, B.Cu at (164.3, 51.1)
- added R110: 2k, Resistor_SMD:R_0603_1608Metric_Pad0.98x0.95mm_HandSolder, B.Cu at (170.7, 51.3)
- added R111: 2k, Resistor_SMD:R_0603_1608Metric_Pad0.98x0.95mm_HandSolder, B.Cu at (158.0, 78.5)
- added R112: 2k, Resistor_SMD:R_0603_1608Metric_Pad0.98x0.95mm_HandSolder, B.Cu at (162.6, 78.5)
- added R113: 2k, Resistor_SMD:R_0603_1608Metric_Pad0.98x0.95mm_HandSolder, B.Cu at (167.6, 78.5)
- added R114: 0, Resistor_SMD:R_0603_1608Metric_Pad0.98x0.95mm_HandSolder, F.Cu at (119.4, 120.1)
- added R115: 0, Resistor_SMD:R_0603_1608Metric_Pad0.98x0.95mm_HandSolder, F.Cu at (110.5, 146.3)
- added R116: 0, Resistor_SMD:R_0603_1608Metric_Pad0.98x0.95mm_HandSolder, F.Cu at (106.4, 143.8)
- added R89: 100, Resistor_SMD:R_0603_1608Metric_Pad0.98x0.95mm_HandSolder, B.Cu at (140.5, 96.5)
- added R90: 100k, Resistor_SMD:R_0603_1608Metric_Pad0.98x0.95mm_HandSolder, F.Cu at (41.9, 70.6)
- added R91: 100, Resistor_SMD:R_0603_1608Metric_Pad0.98x0.95mm_HandSolder, F.Cu at (53.1, 75.2)
- added R92: 100k, Resistor_SMD:R_0603_1608Metric_Pad0.98x0.95mm_HandSolder, B.Cu at (30.7, 90.7)
- added R93: 100, Resistor_SMD:R_0603_1608Metric_Pad0.98x0.95mm_HandSolder, F.Cu at (43.4, 89.7)
- added R94: 100k, Resistor_SMD:R_0603_1608Metric_Pad0.98x0.95mm_HandSolder, B.Cu at (63.0, 90.7)
- added R95: 100, Resistor_SMD:R_0603_1608Metric_Pad0.98x0.95mm_HandSolder, F.Cu at (51.3, 89.8)
- added R96: 2k, Resistor_SMD:R_0603_1608Metric_Pad0.98x0.95mm_HandSolder, F.Cu at (117.1, 93.9)
- added R97: 2k, Resistor_SMD:R_0603_1608Metric_Pad0.98x0.95mm_HandSolder, F.Cu at (132.6, 93.5)
- added R98: 2k, Resistor_SMD:R_0603_1608Metric_Pad0.98x0.95mm_HandSolder, F.Cu at (101.0, 79.0)
- added R99: 2k, Resistor_SMD:R_0603_1608Metric_Pad0.98x0.95mm_HandSolder, B.Cu at (100.1, 92.7)
- added TP10: L_Bass, ECE445L:Testpoint_1x02_P2.54mm, F.Cu at (131.3, 36.1)
- added TP5: R_Treble, ECE445L:Testpoint_1x02_P2.54mm, F.Cu at (132.1, 84.8)
- added TP6: R_Mid, ECE445L:Testpoint_1x02_P2.54mm, F.Cu at (107.2, 93.7)
- added TP7: R_Bass, ECE445L:Testpoint_1x02_P2.54mm, F.Cu at (116.3, 64.0)
- added TP8: L_Treble, ECE445L:Testpoint_1x02_P2.54mm, F.Cu at (175.3, 56.6)
- added TP9: L_Mid, ECE445L:Testpoint_1x02_P2.54mm, F.Cu at (146.8, 47.7)
- C10, C8, C9: value 0.1uF -> 0.1u
- C15, C17, C26, C37, R10, R11, R12, R14, R39, R56, R61, R62, R8: moved to F.Cu
- C18, R15, R20, R21, R23, R28, R29, R3, R37, R4, R44, R46, R5, R52, R53, R58, R86: moved to B.Cu
- C4: value 0.01uF -> 0.1u; moved to B.Cu
- C5: value 0.1uF -> 0.1u; moved to B.Cu
- C6: value 1uF -> 0.1u; moved to B.Cu
- C7: value 2.2uF -> 0.1u; footprint Capacitor_SMD:C_1206_3216Metric_Pad1.33x1.80mm_HandSolder -> Capacitor_SMD:C_0603_1608Metric_Pad1.08x0.95mm_HandSolder
- Q1: value PZT2222A -> MMBF170; footprint Package_TO_SOT_SMD:SOT-223-3_TabPin2 -> Package_TO_SOT_SMD:SOT-23-3; moved to F.Cu
- Q10, Q13, Q15, Q4: value PZT2222A -> MMBF170; footprint Package_TO_SOT_SMD:SOT-223-3_TabPin2 -> Package_TO_SOT_SMD:SOT-23-3; moved to B.Cu
- Q11, Q12, Q14, Q16, Q17, Q18, Q2, Q3, Q5, Q6, Q7, Q8, Q9: value PZT2222A -> MMBF170; footprint Package_TO_SOT_SMD:SOT-223-3_TabPin2 -> Package_TO_SOT_SMD:SOT-23-3
- R6: value 1M -> 0
- R70, R71: value 10k -> 100k; moved to B.Cu
- R72, R74: value 10k -> 100
- R73, R75: value 10k -> 100k
- R76: value 10k -> 100; moved to F.Cu
- R85: value 2k -> 1.5k
- R88: value 2k -> 1.5V; moved to F.Cu
- TP4: value R_Bass -> GND
- U5: value TM4C123GH6PMIR -> FT232R; footprint ECE445L:QFP50P1200X1200X160-64N -> ECE445L:FT232R-Breakout
- moved R72 128.3 mm to (155.4, 96.3), turned to 180 degrees
- moved TP4 91.5 mm to (27.9, 53.3), turned to 0 degrees
- moved C7 79.1 mm to (63.8, 62.7), turned to 180 degrees
- moved C6 71.9 mm to (44.2, 62.2), turned to 180 degrees
- moved C8 71.6 mm to (54.0, 77.7), turned to 180 degrees
- moved R6 64.9 mm to (118.4, 67.8), turned to 90 degrees
- moved C5 59.2 mm to (152.1, 91.9), turned to -90 degrees
- moved C10 59.0 mm to (50.5, 92.5), turned to 0 degrees
- moved C9 55.1 mm to (44.2, 92.5), turned to 180 degrees
- moved C4 53.9 mm to (142.0, 91.9), turned to -90 degrees
- moved TP3 38.8 mm to (131.1, 54.1), turned to 0 degrees
- moved R3 36.8 mm to (138.1, 61.0), turned to 180 degrees
- moved R4 35.0 mm to (134.6, 61.0), turned to 180 degrees
- moved U5 33.4 mm to (123.5, 138.4), turned to -90 degrees
- moved R76 32.5 mm to (62.7, 60.2)
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Connections:
- C10 pad 1: +3V3 -> GND
- C10 pad 2: GND -> PE5
- C4 pad 1: +3V3 -> GND
- C4 pad 2: GND -> PF0
- C5 pad 1: +3V3 -> GND
- C5 pad 2: GND -> PF1
- C6 pad 1: /Lab7_microcontroller/LDO -> GND
- C6 pad 2: GND -> PF2
- C7 pad 1: /Lab7_microcontroller/LDO -> GND
- C7 pad 2: GND -> PF3
- C8 pad 1: /Lab7_microcontroller/LDO -> GND
- C8 pad 2: GND -> PF4
- C9 pad 1: /Lab7_microcontroller/LDO -> GND
- C9 pad 2: GND -> PC7
- D1 pad 1: GND -> PD6
- D2 pad 1: GND -> PD7
- J2 pad J1_1: +3V3 -> Net-(J2-+3.3V)
- J2 pad J3_1: unconnected-(J2-+VBUS-PadJ3_1) -> Net-(J2-+VBUS)
- Q1 pad 1: PB6 -> Net-(Q1-B)
- Q10 pad 1: PB6 -> Net-(Q10-B)
- Q11 pad 1: PB2 -> Net-(Q11-B)
- Q12 pad 1: PB7 -> Net-(Q12-B)
- Q13 pad 1: PB3 -> Net-(Q13-B)
- Q14 pad 1: PB4 -> Net-(Q14-B)
- Q15 pad 1: PB5 -> Net-(Q15-B)
- Q16 pad 1: PC4 -> Net-(Q16-B)
- Q17 pad 1: PC5 -> Net-(Q17-B)
- Q18 pad 1: PC6 -> Net-(Q18-B)
- Q2 pad 1: PB2 -> Net-(Q2-B)
- Q3 pad 1: PB7 -> Net-(Q3-B)
- Q4 pad 1: PB3 -> Net-(Q4-B)
- Q5 pad 1: PB4 -> Net-(Q5-B)
- Q6 pad 1: PB5 -> Net-(Q6-B)
- Q7 pad 1: PC4 -> Net-(Q7-B)
- Q8 pad 1: PC5 -> Net-(Q8-B)
- Q9 pad 1: PC6 -> Net-(Q9-B)
- R46 pad 1: Net-(Q12-C) -> Net-(U11A--)
- R46 pad 2: Net-(U11A--) -> Net-(Q12-C)
- R47 pad 1: Net-(Q13-C) -> Net-(U12A--)
- R47 pad 2: Net-(U12A--) -> Net-(Q13-C)
- R53 pad 1: Net-(Q15-C) -> Net-(U13A--)
- R53 pad 2: Net-(U13A--) -> Net-(Q15-C)
- R6 pad 1: +3V3 -> PD0
- R6 pad 2: Net-(U5-~{WAKE}) -> R_Bass
- R70 pad 2: PF0 -> /Lab7_Input/Pause
- R71 pad 2: PF1 -> /Lab7_Input/LCDMode
- R72 pad 1: +3V3 -> /Lab7_Input/LCDMode
- R72 pad 2: PF2 -> PF1
- R73 pad 2: PF3 -> /Lab7_Input/Flanger
- R74 pad 1: +3V3 -> /Lab7_Input/Flanger
- R74 pad 2: PF4 -> PF2
- R75 pad 2: PC7 -> /Lab7_Input/Distortion
- R76 pad 1: +3V3 -> /Lab7_Input/Distortion
- R76 pad 2: PE5 -> PF3
- R85 pad 1: PD6 -> +3V3
- R88 pad 1: PD7 -> +3V3
- SW2 pad 2: PF0 -> /Lab7_Input/Pause
- SW3 pad 2: PF1 -> /Lab7_Input/LCDMode
- SW4 pad 2: PF2 -> /Lab7_Input/Flanger
- SW5 pad 2: PF3 -> /Lab7_Input/Distortion
- SW6 pad 2: PF4 -> /Lab7_Input/Reverb
- SW7 pad 2: PC7 -> /Lab7_Input/Delay
- SW8 pad 2: PE5 -> /Lab7_Input/Tempo
- TP4 pad 1: R_Bass -> GND
- TP4 pad 2: R_Bass -> GND
- U5 pad 1: PB6 -> Net-(U5A-3V3)
- U5 pad 10: PD7 -> unconnected-(U5B-CTS-Pad10)
- U5 pad 11: +3V3 -> unconnected-(U5B-SLEEP-Pad11)
- U5 pad 12: GND -> unconnected-(U5B-TXDEN-Pad12)
- U5 pad 13: PC7 -> unconnected-(U5B-PWREN-Pad13)
- U5 pad 14: PC6 -> unconnected-(U5B-TXD-Pad14)
- U5 pad 15: PC5 -> unconnected-(U5B-DTR-Pad15)
- U5 pad 16: PC4 -> unconnected-(U5B-RTS-Pad16)
- U5 pad 17: PA0 -> unconnected-(U5B-VCCIO-Pad17)
- U5 pad 18: PA1 -> unconnected-(U5B-RXD-Pad18)
- U5 pad 19: PA2 -> unconnected-(U5B-RI-Pad19)
- U5 pad 2: +3V3 -> ESP_IN_USB_OUT
- U5 pad 20: PA3 -> unconnected-(U5B-GND-Pad20)
- U5 pad 21: PA4 -> unconnected-(U5B-DSR-Pad21)
- U5 pad 22: PA5 -> unconnected-(U5B-DCD-Pad22)
- U5 pad 3: GND -> ESP_OUT_USB_IN
- U5 pad 4: PB7 -> GND
- U5 pad 5: PF4 -> unconnected-(U5B-GND-Pad5)
- U5 pad 6: PE3 -> unconnected-(U5B-TXLED-Pad6)
- U5 pad 7: PE2 -> unconnected-(U5B-RXLED-Pad7)
- U5 pad 8: PE1 -> unconnected-(U5B-VCC-Pad8)
- U5 pad 9: PE0 -> unconnected-(U5B-3v3-Pad9)
Routing:
- net +VRail: track 72.2 -> 271.3 mm, vias 1 -> 5
- net PB0: track 297.9 -> 150.1 mm, vias 8 -> 5
- net PB3: track 230.3 -> 122.7 mm, vias 9 -> 6
- net PC6: track 204.7 -> 129.2 mm, vias 7 -> 5
- net PF4: track 130.4 -> 55.6 mm, vias 4 -> 1
- net ESP_OUT_USB_IN: track 74.4 -> 143.2 mm, vias 4 -> 5
- net ESP_IN_USB_OUT: track 73.2 -> 140.8 mm, vias 4 -> 3
- net PB5: track 213.8 -> 147.9 mm, vias 10 -> 5
- net /Lab7_microcontroller/TDI: track 64.3 -> 0.00 mm, vias 1 -> 0
- net /Lab7_microcontroller/LDO: track 63.0 -> 0.00 mm, vias 2 -> 0
- net /Lab7_microcontroller/TCK: track 62.4 -> 0.00 mm, vias 1 -> 0
- net PA3: track 131.2 -> 69.3 mm
- net /Lab7_microcontroller/TMS: track 59.6 -> 0.00 mm, vias 1 -> 0
- net PB4: track 299.0 -> 240.0 mm
- net /Lab7_microcontroller/TDO: track 58.2 -> 0.00 mm, vias 1 -> 0
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Other:
- board text added: "Power Switch"
