File: hw/ECE445L_Lab7/ECE445L_Lab7.kicad_sch (KiCad schematic)
At the start: 4 parts

Commit message: Created spice models for analog circuits, started kicad schematic -> right audio channel, screen, basic power
Other:
- sheet Lab7_wifi renamed Lab7_analog
- sheet Lab7_analog: file Lab7_wifi.kicad_sch -> Lab7_analog.kicad_sch
Changed lines of the file:
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@@
 (kicad_sch
-	(version 20231120)
+	(version 20250114)
 	(generator "eeschema")
-	(generator_version "8.0")
+	(generator_version "9.0")
 	(paper "A4")
 	(title_block
@@
 		(at 38.1 25.4)
 		(size 196.85 20.955)
+		(exclude_from_sim no)
+		(in_bom yes)
+		(on_board yes)
+		(dnp no)
 		(fields_autoplaced yes)
 		(stroke
@@
 		)
 		(instances
-			(project "Lab7"
+			(project "ECE445L_Lab7"
 				(path "/69b823fd-c065-40ff-9bb9-c5835555f3eb"
 					(page "2")
@@
 		(at 169.545 102.87)
 		(size 35.56 16.51)
+		(exclude_from_sim no)
+		(in_bom yes)
+		(on_board yes)
+		(dnp no)
 		(fields_autoplaced yes)
 		(stroke
@@
 			(color 255 229 191 1.0000)
 		)
-		(property "Sheetname" "Lab7_wifi"
+		(property "Sheetname" "Lab7_analog"
 			(at 169.545 102.1584 0)
 			(effects
@@
 			)
 		)
-		(property "Sheetfile" "Lab7_wifi.kicad_sch"
+		(property "Sheetfile" "Lab7_analog.kicad_sch"
 			(at 169.545 119.9646 0)
 			(effects
@@
 		)
 		(instances
-			(project "Lab7"
+			(project "ECE445L_Lab7"
 				(path "/69b823fd-c065-40ff-9bb9-c5835555f3eb"
 					(page "5")
@@
 		(at 186.055 63.5)
 		(size 40.005 19.685)
+		(exclude_from_sim no)
+		(in_bom yes)
+		(on_board yes)
+		(dnp no)
 		(fields_autoplaced yes)
 		(stroke
@@
 		)
 		(instances
-			(project "Lab7"
+			(project "ECE445L_Lab7"
 				(path "/69b823fd-c065-40ff-9bb9-c5835555f3eb"
 					(page "6")
@@
 		(at 104.775 74.295)
 		(size 45.72 21.59)
+		(exclude_from_sim no)
+		(in_bom yes)
+		(on_board yes)
+		(dnp no)
 		(fields_autoplaced yes)
 		(stroke
@@
 		)
 		(instances
-			(project "Lab7"
+			(project "ECE445L_Lab7"
 				(path "/69b823fd-c065-40ff-9bb9-c5835555f3eb"
 					(page "3")
@@
 		(at 39.37 70.485)
 		(size 45.72 25.4)
+		(exclude_from_sim no)
+		(in_bom yes)
+		(on_board yes)
+		(dnp no)
 		(fields_autoplaced yes)
 		(stroke
@@
 		)
 		(instances
-			(project "Lab7"
+			(project "ECE445L_Lab7"
 				(path "/69b823fd-c065-40ff-9bb9-c5835555f3eb"
 					(page "4")
@@
 		)
 	)
+	(embedded_fonts no)
 )

Commit message: Updated hardware schematic
Other:
- added sheet Lab7_LeftAudio (Lab7_LeftAudio.kicad_sch)
Changed lines of the file:
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@@
+	)
+	(sheet
+		(at 210.185 102.87)
+		(size 31.75 17.145)
+		(exclude_from_sim no)
+		(in_bom yes)
+		(on_board yes)
+		(dnp no)
+		(fields_autoplaced yes)
+		(stroke
+			(width 0.1524)
+			(type solid)
+		)
+		(fill
+			(color 248 169 255 1.0000)
+		)
+		(property "Sheetname" "Lab7_LeftAudio"
+			(at 210.185 102.1584 0)
+			(effects
+				(font
+					(size 1.27 1.27)
+				)
+				(justify left bottom)
+			)
+		)
+		(property "Sheetfile" "Lab7_LeftAudio.kicad_sch"
+			(at 210.185 120.5996 0)
+			(effects
+				(font
+					(size 1.27 1.27)
+				)
+				(justify left top)
+			)
+		)
+		(instances
+			(project "ECE445L_Lab7"
+				(path "/69b823fd-c065-40ff-9bb9-c5835555f3eb"
+					(page "7")
+				)
+			)
+		)
 	)
 	(sheet

Commit message: Lab7A Schematic and BOM - Ashton
Connections:
- no-connect marks 0 -> 4
Other:
- sheet Lab7_analog renamed Lab7_RightAudio
- sheet Lab7_RightAudio: file Lab7_analog.kicad_sch -> Lab7_RightAudio.kicad_sch
Changed lines of the file:
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@@
 		(company "The University of Texas at Austin")
+	)
+	(no_connect
+		(at 269.24 46.99)
+	)
+	(no_connect
+		(at 269.24 31.75)
+	)
+	(no_connect
+		(at 269.24 39.37)
+	)
+	(no_connect
+		(at 269.24 24.13)
 	)
 	(symbol
 		(lib_id "ECE445L:MountingHole")
-		(at 272.415 38.735 0)
+		(at 269.24 24.13 0)
 		(unit 1)
 		(exclude_from_sim no)
@@
 		(dnp no)
 		(fields_autoplaced yes)
-		(property "Reference" "H4"
-			(at 268.605 35.56 0)
+		(property "Reference" "H1"
+			(at 265.43 19.05 0)
 			(effects
 				(font
@@
 		)
 		(property "Value" "~"
-			(at 268.605 36.83 0)
+			(at 265.43 21.59 0)
 			(effects
 				(font
@@
 		)
 		(property "Footprint" "ECE445L:MountingHole_4_40"
-			(at 272.415 38.735 0)
+			(at 269.24 24.13 0)
 			(effects
 				(font
@@
 		)
 		(property "Datasheet" ""
-			(at 272.415 38.735 0)
+			(at 269.24 24.13 0)
 			(effects
 				(font
@@
 		)
 		(property "Description" "Drill hole for 4-40 screw"
-			(at 272.415 38.735 0)
+			(at 269.24 24.13 0)
 			(effects
 				(font
@@
 		)
 		(instances
-			(project "Lab7"
-				(path "/69b823fd-c065-40ff-9bb9-c5835555f3eb"
-					(reference "H4")
+			(project ""
+				(path "/69b823fd-c065-40ff-9bb9-c5835555f3eb"
+					(reference "H1")
 					(unit 1)
 				)
@@
 	(symbol
 		(lib_id "ECE445L:MountingHole")
-		(at 272.415 23.495 0)
+		(at 269.24 31.75 0)
 		(unit 1)
 		(exclude_from_sim no)
@@
 		(dnp no)
 		(fields_autoplaced yes)
-		(property "Reference" "H1"
-			(at 268.605 20.32 0)
+		(property "Reference" "H2"
+			(at 265.43 27.305 0)
 			(effects
 				(font
@@
 		)
 		(property "Value" "~"
-			(at 268.605 21.59 0)
+			(at 265.43 29.845 0)
 			(effects
 				(font
@@
 		)
 		(property "Footprint" "ECE445L:MountingHole_4_40"
-			(at 272.415 23.495 0)
+			(at 269.24 31.75 0)
 			(effects
 				(font
@@
 		)
 		(property "Datasheet" ""
-			(at 272.415 23.495 0)
+			(at 269.24 31.75 0)
 			(effects
 				(font
@@
 		)
 		(property "Description" "Drill hole for 4-40 screw"
-			(at 272.415 23.495 0)
+			(at 269.24 31.75 0)
 			(effects
 				(font
@@
 			(project ""
 				(path "/69b823fd-c065-40ff-9bb9-c5835555f3eb"
-					(reference "H1")
+					(reference "H2")
 					(unit 1)
 				)
@@
 	(symbol
 		(lib_id "ECE445L:MountingHole")
-		(at 272.415 28.575 0)
+		(at 269.24 39.37 0)
 		(unit 1)
 		(exclude_from_sim no)
@@
 		(dnp no)
 		(fields_autoplaced yes)
-		(property "Reference" "H2"
-			(at 268.605 25.4 0)
+		(property "Reference" "H3"
+			(at 265.43 34.29 0)
 			(effects
 				(font
@@
 		)
 		(property "Value" "~"
-			(at 268.605 26.67 0)
+			(at 265.43 36.83 0)
 			(effects
 				(font
@@
 		)
 		(property "Footprint" "ECE445L:MountingHole_4_40"
-			(at 272.415 28.575 0)
+			(at 269.24 39.37 0)
 			(effects
 				(font
@@
 		)
 		(property "Datasheet" ""
-			(at 272.415 28.575 0)
+			(at 269.24 39.37 0)
 			(effects
 				(font
@@
 		)
 		(property "Description" "Drill hole for 4-40 screw"
-			(at 272.415 28.575 0)
+			(at 269.24 39.37 0)
 			(effects
 				(font
@@
 		)
 		(instances
-			(project "Lab7"
-				(path "/69b823fd-c065-40ff-9bb9-c5835555f3eb"
-					(reference "H2")
+			(project ""
+				(path "/69b823fd-c065-40ff-9bb9-c5835555f3eb"
+					(reference "H3")
 					(unit 1)
 				)
@@
 	(symbol
 		(lib_id "ECE445L:MountingHole")
-		(at 272.415 33.655 0)
+		(at 269.24 46.99 0)
 		(unit 1)
 		(exclude_from_sim no)
@@
 		(dnp no)
 		(fields_autoplaced yes)
-		(property "Reference" "H3"
-			(at 268.605 30.48 0)
+		(property "Reference" "H4"
+			(at 265.43 41.91 0)
 			(effects
 				(font
@@
 		)
 		(property "Value" "~"
-			(at 268.605 31.75 0)
+			(at 265.43 44.45 0)
 			(effects
 				(font
@@
 		)
 		(property "Footprint" "ECE445L:MountingHole_4_40"
-			(at 272.415 33.655 0)
+			(at 269.24 46.99 0)
 			(effects
 				(font
@@
 		)
 		(property "Datasheet" ""
-			(at 272.415 33.655 0)
+			(at 269.24 46.99 0)
 			(effects
 				(font
@@
 		)
 		(property "Description" "Drill hole for 4-40 screw"
-			(at 272.415 33.655 0)
+			(at 269.24 46.99 0)
 			(effects
 				(font
@@
 		)
 		(instances
-			(project "Lab7"
-				(path "/69b823fd-c065-40ff-9bb9-c5835555f3eb"
-					(reference "H3")
+			(project ""
+				(path "/69b823fd-c065-40ff-9bb9-c5835555f3eb"
+					(reference "H4")
 					(unit 1)
 				)
@@
 			(project "ECE445L_Lab7"
 				(path "/69b823fd-c065-40ff-9bb9-c5835555f3eb"
-					(page "7")
+					(page "5")
 				)
 			)
@@
 			(color 255 229 191 1.0000)
 		)
-		(property "Sheetname" "Lab7_analog"
+		(property "Sheetname" "Lab7_RightAudio"
 			(at 169.545 102.1584 0)
 			(effects
@@
 			)
 		)
-		(property "Sheetfile" "Lab7_analog.kicad_sch"
+		(property "Sheetfile" "Lab7_RightAudio.kicad_sch"
 			(at 169.545 119.9646 0)
 			(effects
@@
 			(project "ECE445L_Lab7"
 				(path "/69b823fd-c065-40ff-9bb9-c5835555f3eb"
-					(page "5")
+					(page "4")
 				)
 			)
@@
 			(project "ECE445L_Lab7"
 				(path "/69b823fd-c065-40ff-9bb9-c5835555f3eb"
-					(page "6")
+					(page "7")
 				)
 			)
@@
 			(project "ECE445L_Lab7"
 				(path "/69b823fd-c065-40ff-9bb9-c5835555f3eb"
-					(page "4")
-				)
-			)
+					(page "6")
+				)
+			)

Commit message: Final PCB commit
Other:
- note added: "Please note, some changes were made since lab7a report due to feedback making some current calculations incorrect. This will be corrected."
Changed lines of the file:
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@@
 		(comment 1 "Drawn By Ashton Knecht - atk836")
+	)
+	(text "Please note, some changes were made since lab7a report due to feedback\nmaking some current calculations incorrect. This will be corrected."
+		(exclude_from_sim no)
+		(at 229.87 162.56 0)
+		(effects
+			(font
+				(size 1.27 1.27)
+			)
+		)
 	)
 	(no_connect
