File: hw/ECE445L_Lab7/Lab7_Input.kicad_sch (KiCad schematic)
At the start: 36 parts, among them SW2 Pause, SW3 LCDMode, SW4 Flanger, SW5 Distortion, SW6 Reverb, SW7 Delay, SW8 Tempo

Commit message: Pushing so i can work on my desktop
Other:
- note added: "Flanger Delay Knob"
- note added: "Flanger Frequency Knob"
- note removed: "Distortion Knob"
- note removed: "Flanger Knob"
Changed lines of the file:
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@@
 		)
 	)
-	(text "Distortion\nKnob"
+	(text "Flanger\nDelay\nKnob"
 		(exclude_from_sim no)
 		(at 170.815 18.415 0)
@@
 		)
 	)
-	(text "Flanger\nKnob"
+	(text "Flanger\nFrequency\nKnob "
 		(exclude_from_sim no)
 		(at 147.32 17.78 0)

Commit message: Final PCB commit
Parts:
- renumbered C4 to C28, C5 to C29, C6 to C30, C7 to C31, C8 to C32, C9 to C33, C10 to C34, R70 to R73, R89 to R74, R71 to R75, R72 to R76, R73 to R77, R74 to R78, R75 to R79, R76 to R80, R90 to R81, R91 to R82, R77 to R83, R92 to R84, R93 to R85, R78 to R86, R79 to R87, R94 to R88, R95 to R89, R80 to R90, R81 to R91, R82 to R92, R83 to R93, R84 to R94
