File: hw/ECE445L_Lab7/Lab7_RightAudio.kicad_sch (KiCad schematic)
At the start: 60 parts, among them Q10 PZT2222A, Q11 PZT2222A, Q12 PZT2222A, Q13 PZT2222A, Q14 PZT2222A, Q15 PZT2222A, Q16 PZT2222A, Q17 PZT2222A, Q18 PZT2222A, U11 OPA2350, U12 OPA2350, U13 OPA2350, U15 TLV5616, U6 OPA2350

Commit message: Lab7A Schematic and BOM - Ashton
Parts:
- removed C27, C28: 27n, Capacitor_SMD:C_0805_2012Metric, symbol ECE445L:C
- removed C29: 10n, Capacitor_SMD:C_0805_2012Metric, symbol ECE445L:C
- removed C30: 3.5n, Capacitor_SMD:C_0805_2012Metric, symbol ECE445L:C
- removed C31, C32: 1.2n, Capacitor_SMD:C_0805_2012Metric, symbol ECE445L:C
- removed C33, C35, C36: .1u, Capacitor_SMD:C_0805_2012Metric, symbol ECE445L:C
- removed C34: 0.1u, Capacitor_SMD:C_0805_2012Metric, symbol ECE445L:C
- removed C37: 0.1u, ECE445L:C_Axial_200mil, symbol ECE445L:C
- removed C40: 10u, Capacitor_SMD:C_0805_2012Metric, symbol ECE445L:C
- removed Q10, Q11, Q12, Q13, Q14, Q15, Q16, Q17, Q18: PZT2222A, Package_TO_SOT_SMD:SOT-223-3_TabPin2, symbol Transistor_BJT:PZT2222A
- removed R29, R30, R31, R32, R36, R37, R38, R40, R41, R42, R46, R47, R48: 10k, Resistor_SMD:R_0805_2012Metric, symbol Device:R
- removed R33, R39, R45: 20k, Resistor_SMD:R_0805_2012Metric, symbol Device:R
- removed R34, R35, R43, R44, R51, R52, R53, R54, R55, R56: 100k, Resistor_SMD:R_0805_2012Metric, symbol Device:R
- removed R49, R50: 200k, Resistor_SMD:R_0805_2012Metric, symbol Device:R
- removed R57: 75K, Resistor_SMD:R_0805_2012Metric, symbol Device:R
- removed TP10: L_Treble, ECE445L:Testpoint_1x02_P2.54mm, symbol ECE445L:Testpoint
- removed TP11: L_Buff, ECE445L:Testpoint_1x02_P2.54mm, symbol ECE445L:Testpoint
- removed TP12: L_Out, ECE445L:Testpoint_1x02_P2.54mm, symbol ECE445L:Testpoint
- removed TP8: L_Bass, ECE445L:Testpoint_1x02_P2.54mm, symbol ECE445L:Testpoint
- removed TP9: L_Mid, ECE445L:Testpoint_1x02_P2.54mm, symbol ECE445L:Testpoint
- removed U11, U12, U13, U6: OPA2350, ECE445L:DIP-8_W7.62mm_LongPads, symbol ECE445L:OPA2350
- removed U15: TLV5616, ECE445L:DIP-8_W7.62mm_LongPads, symbol ECE445L:TLV5616
- added C15, C16: 27n, Capacitor_SMD:C_0805_2012Metric, symbol ECE445L:C
- added C17: 10n, Capacitor_SMD:C_0805_2012Metric, symbol ECE445L:C
- added C18: 3.5n, Capacitor_SMD:C_0805_2012Metric, symbol ECE445L:C
- added C19, C20: 1.2n, Capacitor_SMD:C_0805_2012Metric, symbol ECE445L:C
- added C21: 10u, Capacitor_SMD:C_0805_2012Metric, symbol ECE445L:C
- added C22, C23, C24, C25: 0.1u, Capacitor_SMD:C_0805_2012Metric, symbol ECE445L:C
- added C26: 0.1u, ECE445L:C_Axial_200mil, symbol ECE445L:C
- added Q1, Q2, Q3, Q4, Q5, Q6, Q7, Q8, Q9: PZT2222A, Package_TO_SOT_SMD:SOT-223-3_TabPin2, symbol Transistor_BJT:PZT2222A
- added R1, R10, R12, R13, R14, R18, R19, R2, R20, R3, R4, R8, R9: 10k, Resistor_SMD:R_0805_2012Metric, symbol Device:R
- added R11, R17, R5: 20k, Resistor_SMD:R_0805_2012Metric, symbol Device:R
- added R15, R16, R23, R24, R25, R26, R27, R28, R6, R7: 100k, Resistor_SMD:R_0805_2012Metric, symbol Device:R
- added R21, R22: 200k, Resistor_SMD:R_0805_2012Metric, symbol Device:R
- added R77, R83: 0, symbol Device:R
- added R82: 75K, Resistor_SMD:R_0805_2012Metric, symbol Device:R
- added TP3: R_Bass, ECE445L:Testpoint_1x02_P2.54mm, symbol ECE445L:Testpoint
- added TP4: R_Mid, ECE445L:Testpoint_1x02_P2.54mm, symbol ECE445L:Testpoint
- added TP5: R_Treble, ECE445L:Testpoint_1x02_P2.54mm, symbol ECE445L:Testpoint
- added TP6: R_Buff, ECE445L:Testpoint_1x02_P2.54mm, symbol ECE445L:Testpoint
- added TP7: R_Out, ECE445L:Testpoint_1x02_P2.54mm, symbol ECE445L:Testpoint
- added U10, U14, U8, U9: OPA2350, ECE445L:DIP-8_W7.62mm_LongPads, symbol ECE445L:OPA2350
- added U5: TLV5616, ECE445L:DIP-8_W7.62mm_LongPads, symbol ECE445L:TLV5616
Connections:
- net +3V3: now also C22.2, C23.2, C24.2, C25.2, C26.1, R15.2, R21.2, R24.2, R6.2, U10.8 (V+), U14.8 (V+), U5.8 (VDD), U8.8 (V+), U9.8 (V+)
- net GND: now also C16.2, C18.1, C22.1, C23.1, C24.1, C25.1, C26.2, Q1.3 (E), Q2.3 (E), Q3.3 (E), Q4.3 (E), Q5.3 (E), Q6.3 (E), R16.1, R22.1, R25.1, R7.1, U10.4 (V-), U14.4 (V-), U5.3 (~{CS}), U5.5 (AGND), U8.4 (V-), U9.4 (V-)
- net PB2: now also Q1.1 (B)
- net PB3: now also Q2.1 (B)
- net PB4: now also Q3.1 (B)
- net PB5: now also Q4.1 (B)
- net PB6: now also Q5.1 (B)
- net PB7: now also Q6.1 (B)
- net PC4: now also Q7.1 (B)
- net PC5: now also Q8.1 (B)
- net PC6: now also Q9.1 (B)
- net R_Bass: now also R20.1, R83.1, TP3.1 (A), TP3.2 (B), U8.6 (-), U8.7
- net R_Mid: now also R19.1, TP4.1 (A), TP4.2 (B), U9.6 (-), U9.7
- net R_Treble: now also R18.1, TP5.1 (A), TP5.2 (B), U10.6 (-), U10.7
- net VRef: now also U5.6 (REF)
- net Vin: now also C17.1, C19.1
- net Vin_L: now also R1.2
- new net: Q4.2 (C), R10.1
- new net: R10.2, R11.1, R9.1, U9.2 (-)
- new net: C15.1, R4.2, U8.1, U8.5 (+)
- new net: R12.1, R13.2, U10.1, U10.5 (+)
- new net: C19.2, C20.1, R12.2
- new net: C18.2, R8.2, U9.5 (+)
- new net: Q7.2 (C), R26.1, R27.1
- new net: Q3.2 (C), R11.2
- new net: R8.1, R9.2, U9.1
- new net: C17.2, U9.3 (+)
- new net: R3.2, R4.1, R5.1, U8.2 (-)
- new net: Q1.2 (C), R5.2
- new net: C15.2, R1.1, R2.1
- new net: R24.1, R25.2, U14.5 (+)
- new net: R23.2, R26.2, R27.2, R28.2, R82.2, U14.6 (-)
- new net: Q8.2 (C), R82.1
- new net: C16.1, R2.2, U8.3 (+)
- new net: C20.2, R15.1, R16.2, U10.3 (+)
- new net: Q6.2 (C), R14.1
- new net: R13.1, R14.2, R17.1, U10.2 (-)
- new net: R18.2, R19.2, R20.2, U14.3 (+)
- new net: Q2.2 (C), R3.1
- new net: C21.2, R21.1, R22.2, R23.1
- new net: R6.1, R7.2
- new net: Q9.2 (C), R28.1
- new net: Q5.2 (C), R17.2
- new net PD0: R77.1, R83.2
- new net RAUDIO_CLK: U5.2 (SCLK)
- new net RAUDIO_FS: U5.4 (FS)
- new net RAUDIO_OUT: U5.1 (DIN)
- new net R_AudioOut: Q7.3 (E), Q8.3 (E), Q9.3 (E), R77.2, TP7.1 (A), TP7.2 (B), U14.7
- new net R_Buff: C21.1, TP6.1 (A), TP6.2 (B), U14.1, U14.2 (-)
- new net Vin_R: U5.7 (OUT)
Other:
- note added: "Bass In for visulizer"

Commit message: Made changers to the schematic, updated bom, and created priliminary layout for the PCB. Ready for 7B Prep!
Parts:
- C15, C16, C17, C18, C19, C20, C22, C23, C24, C25: footprint Capacitor_SMD:C_0805_2012Metric -> Capacitor_SMD:C_0603_1608Metric
- C26: footprint ECE445L:C_Axial_200mil -> Capacitor_SMD:C_0603_1608Metric
- R1, R10, R11, R12, R13, R14, R15, R16, R17, R18, R19, R2, R20, R21, R22, R23, R24, R25, R26, R27, R28, R3, R4, R5, R6, R7, R8, R82, R9: footprint Resistor_SMD:R_0805_2012Metric -> Resistor_SMD:R_0603_1608Metric
- R77, R83: footprint (none) -> Resistor_SMD:R_0603_1608Metric
Connections:
- net Vin is gone; now on net Vin_R: C17.1, C19.1
- net Vin_L is gone; now on net Vin_R: R1.2
- net +3V3: now also R24.1; no longer R24.2
- net at R25.2, U14.5 (+): now also R24.2; no longer R24.1
Other:
- moved on the sheet: R24
Changed lines of the file:
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@@
 	)
 	(junction
+		(at 226.695 112.395)
+		(diameter 0)
+		(color 0 0 0 0)
+	)
+	(junction
 		(at 60.325 163.83)
 		(diameter 0)
@@
 	)
 	(junction
-		(at 226.695 112.395)
-		(diameter 0)
-		(color 0 0 0 0)
-	)
-	(junction
 		(at 247.015 146.05)
 		(diameter 0)
@@
 	(wire
 		(pts
-			(xy 226.695 109.855) (xy 226.695 112.395)
-		)
-		(stroke
-			(width 0)
-			(type default)
-		)
-	)
-	(wire
-		(pts
 			(xy 92.71 104.775) (xy 92.71 107.315)
 		)
@@
 	(wire
 		(pts
+			(xy 226.695 99.695) (xy 226.695 102.235)
+		)
+		(stroke
+			(width 0)
+			(type default)
+		)
+	)
+	(wire
+		(pts
 			(xy 271.78 158.75) (xy 259.715 158.75)
 		)
@@
 	(wire
 		(pts
-			(xy 226.695 99.695) (xy 226.695 102.235)
-		)
-		(stroke
-			(width 0)
-			(type default)
-		)
-	)
-	(wire
-		(pts
 			(xy 99.06 104.775) (xy 104.14 104.775)
 		)
@@
 	(wire
 		(pts
+			(xy 226.695 109.855) (xy 226.695 112.395)
+		)
+		(stroke
+			(width 0)
+			(type default)
+		)
+	)
+	(wire
+		(pts
 			(xy 267.97 142.875) (xy 267.97 139.065)
 		)
@@
 		)
 	)
-	(global_label "Vin"
+	(global_label "Vin_R"
 		(shape input)
 		(at 70.485 92.075 180)
@@
 		)
 		(property "Intersheetrefs" "${INTERSHEET_REFS}"
-			(at 64.6574 92.075 0)
+			(at 62.4198 92.075 0)
 			(effects
 				(font
@@
 		)
 	)
-	(global_label "Vin"
+	(global_label "Vin_R"
 		(shape input)
 		(at 20.955 38.1 180)
@@
 		)
 		(property "Intersheetrefs" "${INTERSHEET_REFS}"
-			(at 15.1274 38.1 0)
+			(at 12.8898 38.1 0)
 			(effects
 				(font
@@
 		)
 	)
-	(global_label "Vin_L"
+	(global_label "Vin_R"
 		(shape input)
 		(at 21.59 151.765 180)
@@
 		)
 		(property "Intersheetrefs" "${INTERSHEET_REFS}"
-			(at 13.7667 151.765 0)
+			(at 13.5248 151.765 0)
 			(effects
 				(font
@@
 			)
 		)
-		(property "Footprint" "Capacitor_SMD:C_0805_2012Metric"
+		(property "Footprint" "Capacitor_SMD:C_0603_1608Metric"
 			(at 167.9448 27.94 0)
 			(effects
@@
 			)
 		)
-		(property "Footprint" "Capacitor_SMD:C_0805_2012Metric"
+		(property "Footprint" "Capacitor_SMD:C_0603_1608Metric"
 			(at 148.8948 29.21 0)
 			(effects
@@
 			)
 		)
-		(property "Footprint" "Resistor_SMD:R_0805_2012Metric"
+		(property "Footprint" "Resistor_SMD:R_0603_1608Metric"
 			(at 100.838 111.125 90)
 			(effects
@@
 			)
 		)
-		(property "Footprint" "Capacitor_SMD:C_0805_2012Metric"
+		(property "Footprint" "Capacitor_SMD:C_0603_1608Metric"
 			(at 130.4798 29.21 0)
 			(effects
@@
 			)
 		)
-		(property "Footprint" "Resistor_SMD:R_0805_2012Metric"
+		(property "Footprint" "Resistor_SMD:R_0603_1608Metric"
 			(at 31.877 27.305 90)
 			(effects
@@
 			)
 		)
-		(property "Footprint" ""
+		(property "Footprint" "Resistor_SMD:R_0603_1608Metric"
 			(at 100.457 170.18 90)
 			(effects
@@
 			)
 		)
-		(property "Footprint" "Resistor_SMD:R_0805_2012Metric"
+		(property "Footprint" "Resistor_SMD:R_0603_1608Metric"
 			(at 52.197 170.18 90)
 			(effects
@@
 			)
 		)
-		(property "Footprint" "Resistor_SMD:R_0805_2012Metric"
+		(property "Footprint" "Resistor_SMD:R_0603_1608Metric"
 			(at 119.38 96.393 90)
 			(effects
@@
 			)
 		)
-		(property "Footprint" "Capacitor_SMD:C_0805_2012Metric"
+		(property "Footprint" "Capacitor_SMD:C_0603_1608Metric"
 			(at 36.5252 146.685 0)
 			(effects
@@
 			)
 		)
-		(property "Footprint" "Resistor_SMD:R_0805_2012Metric"
+		(property "Footprint" "Resistor_SMD:R_0603_1608Metric"
 			(at 41.275 153.543 90)
 			(effects
@@
 			)
 		)
-		(property "Footprint" "Resistor_SMD:R_0805_2012Metric"
+		(property "Footprint" "Resistor_SMD:R_0603_1608Metric"
 			(at 90.932 111.125 90)
 			(effects
@@
 	(symbol
 		(lib_id "Device:R")
-		(at 226.695 106.045 180)
+		(at 226.695 106.045 0)
 		(unit 1)
 		(exclude_from_sim no)
@@
 		(dnp no)
 		(property "Reference" "R24"
-			(at 224.155 107.95 90)
+			(at 229.235 104.14 90)
 			(effects
 				(font
@@
 		)
 		(property "Value" "100k"
-			(at 226.695 108.585 90)
+			(at 226.695 103.505 90)
 			(effects
 				(font
@@
 			)
 		)
-		(property "Footprint" "Resistor_SMD:R_0805_2012Metric"
-			(at 228.473 106.045 90)
+		(property "Footprint" "Resistor_SMD:R_0603_1608Metric"
+			(at 224.917 106.045 90)
 			(effects
 				(font
@@
 			)
 		)
-		(property "Footprint" "Resistor_SMD:R_0805_2012Metric"
+		(property "Footprint" "Resistor_SMD:R_0603_1608Metric"
 			(at 47.498 33.02 90)
 			(effects
@@
 			)
 		)
-		(property "Footprint" "Resistor_SMD:R_0805_2012Metric"
+		(property "Footprint" "Resistor_SMD:R_0603_1608Metric"
 			(at 61.468 56.515 90)
 			(effects
@@
 			)
 		)
-		(property "Footprint" "Resistor_SMD:R_0805_2012Metric"
+		(property "Footprint" "Resistor_SMD:R_0603_1608Metric"
 			(at 175.26 134.493 90)
 			(effects
@@
 			)
 		)
-		(property "Footprint" ""
+		(property "Footprint" "Resistor_SMD:R_0603_1608Metric"
 			(at 110.49 177.673 90)
 			(effects
@@
 			)
 		)
-		(property "Footprint" "Resistor_SMD:R_0805_2012Metric"
+		(property "Footprint" "Resistor_SMD:R_0603_1608Metric"
 			(at 62.103 170.18 90)
 			(effects
@@
 			)
 		)
-		(property "Footprint" "Resistor_SMD:R_0805_2012Metric"
+		(property "Footprint" "Resistor_SMD:R_0603_1608Metric"
 			(at 175.26 123.698 90)
 			(effects
@@
 			)
 		)
-		(property "Footprint" "Capacitor_SMD:C_0805_2012Metric"
+		(property "Footprint" "Capacitor_SMD:C_0603_1608Metric"
 			(at 47.3202 168.91 0)
 			(effects
@@
 			)
 		)
-		(property "Footprint" "Resistor_SMD:R_0805_2012Metric"
+		(property "Footprint" "Resistor_SMD:R_0603_1608Metric"
 			(at 247.142 150.495 90)
 			(effects
@@
 			)
 		)
-		(property "Footprint" "Resistor_SMD:R_0805_2012Metric"
+		(property "Footprint" "Resistor_SMD:R_0603_1608Metric"
 			(at 47.498 51.435 90)
 			(effects
@@
 			)
 		)
-		(property "Footprint" "Capacitor_SMD:C_0805_2012Metric"
+		(property "Footprint" "Capacitor_SMD:C_0603_1608Metric"
 			(at 32.385 37.1348 0)
 			(effects
@@
 			)
 		)
-		(property "Footprint" "ECE445L:C_Axial_200mil"
+		(property "Footprint" "Capacitor_SMD:C_0603_1608Metric"
 			(at 263.8552 51.435 0)
 			(effects
@@
 			)
 		)
-		(property "Footprint" "Capacitor_SMD:C_0805_2012Metric"
+		(property "Footprint" "Capacitor_SMD:C_0603_1608Metric"
 			(at 44.45 37.1348 0)
 			(effects
@@
 			)
 		)
-		(property "Footprint" "Resistor_SMD:R_0805_2012Metric"
+		(property "Footprint" "Resistor_SMD:R_0603_1608Metric"
 			(at 228.6 126.238 90)
 			(effects
@@
 			)
 		)
-		(property "Footprint" "Resistor_SMD:R_0805_2012Metric"
+		(property "Footprint" "Resistor_SMD:R_0603_1608Metric"
 			(at 86.233 98.425 90)
 			(effects
@@
 			)
 		)
-		(property "Footprint" "Resistor_SMD:R_0805_2012Metric"
+		(property "Footprint" "Resistor_SMD:R_0603_1608Metric"
 			(at 219.583 134.62 90)
 			(effects
@@
 			)
 		)
-		(property "Footprint" "Resistor_SMD:R_0805_2012Metric"
+		(property "Footprint" "Resistor_SMD:R_0603_1608Metric"
 			(at 219.583 105.41 90)
 			(effects
@@
 			)
 		)
-		(property "Footprint" "Resistor_SMD:R_0805_2012Metric"
+		(property "Footprint" "Resistor_SMD:R_0603_1608Metric"
 			(at 233.68 110.617 90)
 			(effects
@@
 			)
 		)
-		(property "Footprint" "Resistor_SMD:R_0805_2012Metric"
+		(property "Footprint" "Resistor_SMD:R_0603_1608Metric"
 			(at 69.215 165.608 90)
 			(effects
@@
 			)
 		)
-		(property "Footprint" "Resistor_SMD:R_0805_2012Metric"
+		(property "Footprint" "Resistor_SMD:R_0603_1608Metric"
 			(at 175.895 112.903 90)
 			(effects
@@
 			)
 		)
-		(property "Footprint" "Capacitor_SMD:C_0805_2012Metric"
+		(property "Footprint" "Capacitor_SMD:C_0603_1608Metric"
 			(at 186.9948 27.94 0)
 			(effects
@@
 			)
 		)
-		(property "Footprint" "Resistor_SMD:R_0805_2012Metric"
+		(property "Footprint" "Resistor_SMD:R_0603_1608Metric"
 			(at 243.332 150.495 90)
 			(effects
@@
 			)
 		)
-		(property "Footprint" "Resistor_SMD:R_0805_2012Metric"
+		(property "Footprint" "Resistor_SMD:R_0603_1608Metric"
 			(at 51.562 56.515 90)
 			(effects
@@
 			)
 		)
-		(property "Footprint" "Resistor_SMD:R_0805_2012Metric"
+		(property "Footprint" "Resistor_SMD:R_0603_1608Metric"
 			(at 270.002 150.495 90)
 			(effects
@@
 			)
 		)
-		(property "Footprint" "Resistor_SMD:R_0805_2012Metric"
+		(property "Footprint" "Resistor_SMD:R_0603_1608Metric"
 			(at 68.58 51.943 90)
 			(effects
@@
 			)
 		)
-		(property "Footprint" "Resistor_SMD:R_0805_2012Metric"
+		(property "Footprint" "Resistor_SMD:R_0603_1608Metric"
 			(at 29.21 149.987 90)
 			(effects
@@
 			)
 		)
-		(property "Footprint" "Resistor_SMD:R_0805_2012Metric"
+		(property "Footprint" "Resistor_SMD:R_0603_1608Metric"
 			(at 257.937 150.495 90)
 			(effects
@@
 			)
 		)
-		(property "Footprint" "Capacitor_SMD:C_0805_2012Metric"
+		(property "Footprint" "Capacitor_SMD:C_0603_1608Metric"
 			(at 126.0348 97.79 0)
 			(effects
@@
 			)
 		)
-		(property "Footprint" "Resistor_SMD:R_0805_2012Metric"
+		(property "Footprint" "Resistor_SMD:R_0603_1608Metric"
 			(at 86.233 86.995 90)
 			(effects
@@
 			)
 		)
-		(property "Footprint" "Capacitor_SMD:C_0805_2012Metric"
+		(property "Footprint" "Capacitor_SMD:C_0603_1608Metric"
 			(at 80.645 91.1098 0)
 			(effects
@@
 			)
 		)
-		(property "Footprint" "Resistor_SMD:R_0805_2012Metric"
+		(property "Footprint" "Resistor_SMD:R_0603_1608Metric"
 			(at 107.95 106.553 90)
 			(effects

Commit message: Rough draft layout - need to remove tm4c chip
Parts:
- removed R83: 0, Resistor_SMD:R_0603_1608Metric, symbol Device:R
- removed TP3: R_Bass, ECE445L:Testpoint_1x02_P2.54mm, symbol ECE445L:Testpoint
- removed TP4: R_Mid, ECE445L:Testpoint_1x02_P2.54mm, symbol ECE445L:Testpoint
- removed TP5: R_Treble, ECE445L:Testpoint_1x02_P2.54mm, symbol ECE445L:Testpoint
- removed TP6: R_Buff, ECE445L:Testpoint_1x02_P2.54mm, symbol ECE445L:Testpoint
- removed TP7: R_Out, ECE445L:Testpoint_1x02_P2.54mm, symbol ECE445L:Testpoint
- added R28: 40k, Resistor_SMD:R_0603_1608Metric_Pad0.98x0.95mm_HandSolder, symbol Device:R
- added R29: 3.3k, Resistor_SMD:R_0603_1608Metric_Pad0.98x0.95mm_HandSolder, symbol Device:R
- C15: renamed from C19; footprint Capacitor_SMD:C_0603_1608Metric -> Capacitor_SMD:C_0603_1608Metric_Pad1.08x0.95mm_HandSolder
- C16: renamed from C15; value 27n -> 30n; footprint Capacitor_SMD:C_0603_1608Metric -> Capacitor_SMD:C_0603_1608Metric_Pad1.08x0.95mm_HandSolder
- C17: renamed from C20; footprint Capacitor_SMD:C_0603_1608Metric -> Capacitor_SMD:C_0603_1608Metric_Pad1.08x0.95mm_HandSolder
- C18: renamed from C16; value 27n -> 30n; footprint Capacitor_SMD:C_0603_1608Metric -> Capacitor_SMD:C_0603_1608Metric_Pad1.08x0.95mm_HandSolder
- C19: renamed from C17; value 10n -> 9.5n; footprint Capacitor_SMD:C_0603_1608Metric -> Capacitor_SMD:C_0603_1608Metric_Pad1.08x0.95mm_HandSolder
- C20: renamed from C18; value 3.5n -> 3.7n; footprint Capacitor_SMD:C_0603_1608Metric -> Capacitor_SMD:C_0603_1608Metric_Pad1.08x0.95mm_HandSolder
- C21: renamed from C22; footprint Capacitor_SMD:C_0603_1608Metric -> Capacitor_SMD:C_0603_1608Metric_Pad1.08x0.95mm_HandSolder
- C22: renamed from C23; footprint Capacitor_SMD:C_0603_1608Metric -> Capacitor_SMD:C_0603_1608Metric_Pad1.08x0.95mm_HandSolder
- C23: renamed from C24; footprint Capacitor_SMD:C_0603_1608Metric -> Capacitor_SMD:C_0603_1608Metric_Pad1.08x0.95mm_HandSolder
- C24: renamed from C25; footprint Capacitor_SMD:C_0603_1608Metric -> Capacitor_SMD:C_0603_1608Metric_Pad1.08x0.95mm_HandSolder
- C25: renamed from C21; footprint Capacitor_SMD:C_0805_2012Metric -> Capacitor_SMD:C_0805_2012Metric_Pad1.18x1.45mm_HandSolder
- C26: footprint Capacitor_SMD:C_0603_1608Metric -> Capacitor_SMD:C_0603_1608Metric_Pad1.08x0.95mm_HandSolder
- R10: renamed from R15; footprint Resistor_SMD:R_0603_1608Metric -> Resistor_SMD:R_0603_1608Metric_Pad0.98x0.95mm_HandSolder
- R11: renamed from R16; footprint Resistor_SMD:R_0603_1608Metric -> Resistor_SMD:R_0603_1608Metric_Pad0.98x0.95mm_HandSolder
- R12: renamed from R17; footprint Resistor_SMD:R_0603_1608Metric -> Resistor_SMD:R_0603_1608Metric_Pad0.98x0.95mm_HandSolder
- R13: renamed from R5; footprint Resistor_SMD:R_0603_1608Metric -> Resistor_SMD:R_0603_1608Metric_Pad0.98x0.95mm_HandSolder
- R14: footprint Resistor_SMD:R_0603_1608Metric -> Resistor_SMD:R_0603_1608Metric_Pad0.98x0.95mm_HandSolder
- R15: renamed from R3; footprint Resistor_SMD:R_0603_1608Metric -> Resistor_SMD:R_0603_1608Metric_Pad0.98x0.95mm_HandSolder
- R16: renamed from R13; footprint Resistor_SMD:R_0603_1608Metric -> Resistor_SMD:R_0603_1608Metric_Pad0.98x0.95mm_HandSolder
- R17: renamed from R4; footprint Resistor_SMD:R_0603_1608Metric -> Resistor_SMD:R_0603_1608Metric_Pad0.98x0.95mm_HandSolder
- R18: renamed from R6; footprint Resistor_SMD:R_0603_1608Metric -> Resistor_SMD:R_0603_1608Metric_Pad0.98x0.95mm_HandSolder
- R19: renamed from R7; footprint Resistor_SMD:R_0603_1608Metric -> Resistor_SMD:R_0603_1608Metric_Pad0.98x0.95mm_HandSolder
- R20: renamed from R11; footprint Resistor_SMD:R_0603_1608Metric -> Resistor_SMD:R_0603_1608Metric_Pad0.98x0.95mm_HandSolder
- R21: renamed from R10; footprint Resistor_SMD:R_0603_1608Metric -> Resistor_SMD:R_0603_1608Metric_Pad0.98x0.95mm_HandSolder
- R22: renamed from R9; footprint Resistor_SMD:R_0603_1608Metric -> Resistor_SMD:R_0603_1608Metric_Pad0.98x0.95mm_HandSolder
- R23: renamed from R77; footprint Resistor_SMD:R_0603_1608Metric -> Resistor_SMD:R_0603_1608Metric_Pad0.98x0.95mm_HandSolder
- R24: renamed from R8; footprint Resistor_SMD:R_0603_1608Metric -> Resistor_SMD:R_0603_1608Metric_Pad0.98x0.95mm_HandSolder
- R25: renamed from R19; value 10k -> 7.5k; footprint Resistor_SMD:R_0603_1608Metric -> Resistor_SMD:R_0603_1608Metric_Pad0.98x0.95mm_HandSolder
- R26: renamed from R20; footprint Resistor_SMD:R_0603_1608Metric -> Resistor_SMD:R_0603_1608Metric_Pad0.98x0.95mm_HandSolder
- R27: renamed from R18; footprint Resistor_SMD:R_0603_1608Metric -> Resistor_SMD:R_0603_1608Metric_Pad0.98x0.95mm_HandSolder
- R30: renamed from R21; footprint Resistor_SMD:R_0603_1608Metric -> Resistor_SMD:R_0603_1608Metric_Pad0.98x0.95mm_HandSolder
- R31: renamed from R22; footprint Resistor_SMD:R_0603_1608Metric -> Resistor_SMD:R_0603_1608Metric_Pad0.98x0.95mm_HandSolder
- R32: renamed from R24; footprint Resistor_SMD:R_0603_1608Metric -> Resistor_SMD:R_0603_1608Metric_Pad0.98x0.95mm_HandSolder
- R33: renamed from R23; footprint Resistor_SMD:R_0603_1608Metric -> Resistor_SMD:R_0603_1608Metric_Pad0.98x0.95mm_HandSolder
- R34: renamed from R25; footprint Resistor_SMD:R_0603_1608Metric -> Resistor_SMD:R_0603_1608Metric_Pad0.98x0.95mm_HandSolder
- R35: renamed from R26; footprint Resistor_SMD:R_0603_1608Metric -> Resistor_SMD:R_0603_1608Metric_Pad0.98x0.95mm_HandSolder
- R36: renamed from R27; footprint Resistor_SMD:R_0603_1608Metric -> Resistor_SMD:R_0603_1608Metric_Pad0.98x0.95mm_HandSolder
- R37: renamed from R82; footprint Resistor_SMD:R_0603_1608Metric -> Resistor_SMD:R_0603_1608Metric_Pad0.98x0.95mm_HandSolder
- R38: renamed from R28; footprint Resistor_SMD:R_0603_1608Metric -> Resistor_SMD:R_0603_1608Metric_Pad0.98x0.95mm_HandSolder
- R7: renamed from R1; footprint Resistor_SMD:R_0603_1608Metric -> Resistor_SMD:R_0603_1608Metric_Pad0.98x0.95mm_HandSolder
- R8: renamed from R12; footprint Resistor_SMD:R_0603_1608Metric -> Resistor_SMD:R_0603_1608Metric_Pad0.98x0.95mm_HandSolder
- R9: renamed from R2; footprint Resistor_SMD:R_0603_1608Metric -> Resistor_SMD:R_0603_1608Metric_Pad0.98x0.95mm_HandSolder
- renumbered Q5 to Q1, Q1 to Q2, Q6 to Q3, Q2 to Q4, Q3 to Q5, Q4 to Q6, U5 to U10, U10 to U6, U8 to U6, U8 to U7, U10 to U7, U9 to U8, U14 to U9
Connections:
- net GND: now also R28.1
- net R_Buff: now also R29.2; no longer U9.2 (-)
- net R_Treble: now also R27.2; no longer R27.1
- net at C19.2, U8.3 (+): now also R18.1, R19.2
- net at R25.2, R26.2, U9.3 (+): now also R27.1; no longer R27.2
- new net: R28.2, R29.1, U9.2 (-)
Other:
- company: (none) -> The University of Texas at Austin
- title: (none) -> ECE 445L Lab7
- moved on the sheet: R27
