File: hw/ECE445L_Lab7/Lab7_RightAudio.kicad_sch (KiCad schematic)
At the start: 58 parts, among them Q1 PZT2222A, Q2 PZT2222A, Q3 PZT2222A, Q4 PZT2222A, Q5 PZT2222A, Q6 PZT2222A, Q7 PZT2222A, Q8 PZT2222A, Q9 PZT2222A, U10 TLV5616, U6 OPA2350, U7 OPA2350, U8 OPA2350, U9 OPA2350

Commit message: Added current consumption to schematic
Other:
- note added: "100k Ohm Resistor Dividers : 2 * (0.0165 mA) = 0.033 mA 200k Ohm Resistor Dividers : 1 * 0.00825 = 0.00825 mA 10k Ohm Resitor Dividers : 3 * (0.165 mA) = 0.5 mA 75k Ohm Loads : 1 * (0.044 mA) = 0.044 mA OPA2350s : 8 * (7.5 mA) = 60 mA TLV5616s : 1 * (1.1mA) = 1.1 mA Total : 61.6825 mA"
- note added: "Current per 100k Ohm Resitor Divider +3V3 / (100k + 100k) = 0.0165 mA Current per 200k Ohm Resistor Divider +3V3 / (200k + 200k) = 0.00825 mA Current per 10k Ohm Resitor Divider +3V3 / (10k + 10k) = 0.165 mA Current per 75k Load +3V3 / 75k = 0.044 mA Quiescent Current (Per Amplifier - 2x per chip) 7.5 mA Current Per TLV5616 1.1 mA"
- moved on the sheet: R23
Changed lines of the file:
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@@
 		)
 	)
+	(text "100k Ohm Resistor Dividers : 2 * (0.0165 mA) = 0.033 mA\n200k Ohm Resistor Dividers : 1 * 0.00825 = 0.00825 mA\n10k Ohm Resitor Dividers : 3 * (0.165 mA) = 0.5 mA\n75k Ohm Loads : 1 * (0.044 mA) = 0.044 mA\nOPA2350s : 8 * (7.5 mA) = 60 mA\nTLV5616s : 1 * (1.1mA) = 1.1 mA\n\nTotal : 61.6825 mA"
+		(exclude_from_sim no)
+		(at 118.11 184.15 0)
+		(effects
+			(font
+				(size 1.27 1.27)
+			)
+			(justify left)
+		)
+	)
 	(text "Mid Channel"
 		(exclude_from_sim no)
@@
 		)
 	)
+	(text "Current per 100k Ohm Resitor Divider\n+3V3 / (100k + 100k) = 0.0165 mA\n\nCurrent per 200k Ohm Resistor Divider\n+3V3 / (200k + 200k) = 0.00825 mA\n\nCurrent per 10k Ohm Resitor Divider\n+3V3 / (10k + 10k) = 0.165 mA\n\nCurrent per 75k Load\n+3V3 / 75k = 0.044 mA\n\nQuiescent Current (Per Amplifier - 2x per chip)\n7.5 mA\n\nCurrent Per TLV5616\n1.1 mA\n"
+		(exclude_from_sim no)
+		(at 118.745 155.575 0)
+		(effects
+			(font
+				(size 1.27 1.27)
+			)
+			(justify left)
+		)
+	)
 	(text "Treble Channel"
 		(exclude_from_sim no)
@@
 	(text "Bass In for visulizer"
 		(exclude_from_sim no)
-		(at 116.84 169.545 0)
+		(at 101.6 170.815 0)
 		(effects
 			(font
@@
 	(wire
 		(pts
-			(xy 102.235 175.895) (xy 106.68 175.895)
+			(xy 86.995 177.165) (xy 91.44 177.165)
 		)
 		(stroke
@@
 	(wire
 		(pts
-			(xy 102.235 175.895) (xy 102.235 177.8)
+			(xy 86.995 177.165) (xy 86.995 179.07)
 		)
 		(stroke
@@
 	(wire
 		(pts
-			(xy 114.3 175.895) (xy 118.745 175.895)
+			(xy 99.06 177.165) (xy 103.505 177.165)
 		)
 		(stroke
@@
 	(global_label "PD0"
 		(shape passive)
-		(at 102.235 177.8 270)
+		(at 86.995 179.07 270)
 		(fields_autoplaced yes)
 		(effects
@@
 		)
 		(property "Intersheetrefs" "${INTERSHEET_REFS}"
-			(at 102.235 183.4234 90)
+			(at 86.995 184.6934 90)
 			(effects
 				(font
@@
 	(global_label "R_AudioOut"
 		(shape input)
-		(at 118.745 175.895 0)
+		(at 103.505 177.165 0)
 		(fields_autoplaced yes)
 		(effects
@@
 		)
 		(property "Intersheetrefs" "${INTERSHEET_REFS}"
-			(at 132.3134 175.895 0)
+			(at 117.0734 177.165 0)
 			(effects
 				(font
@@
 	(symbol
 		(lib_id "Device:R")
-		(at 110.49 175.895 90)
+		(at 95.25 177.165 90)
 		(unit 1)
 		(exclude_from_sim no)
@@
 		(dnp no)
 		(property "Reference" "R23"
-			(at 112.395 178.435 90)
+			(at 97.155 179.705 90)
 			(effects
 				(font
@@
 		)
 		(property "Value" "0"
-			(at 111.125 175.895 90)
+			(at 95.885 177.165 90)
 			(effects
 				(font
@@
 		)
 		(property "Footprint" "Resistor_SMD:R_0603_1608Metric_Pad0.98x0.95mm_HandSolder"
-			(at 110.49 177.673 90)
+			(at 95.25 178.943 90)
 			(effects
 				(font
@@
 		)
 		(property "Datasheet" "~"
-			(at 110.49 175.895 0)
+			(at 95.25 177.165 0)
 			(effects
 				(font
@@
 		)
 		(property "Description" "Resistor"
-			(at 110.49 175.895 0)
+			(at 95.25 177.165 0)
 			(effects
 				(font

Commit message: Updated lab7a report
Other:
- note added: "Right Audio Current Consumption Current per 100k Ohm Resitor Divider +3V3 / (100k + 100k) = 0.0165 mA Current per 200k Ohm Resistor Divider +3V3 / (200k + 200k) = 0.00825 mA Current per 10k Ohm Resitor Divider +3V3 / (10k + 10k) = 0.165 mA Current per 75k Load +3V3 / 75k = 0.044 mA Quiescent Current (Per Amplifier - 2x per chip) 7.5 mA Current Per TLV5616 1.1 mA"
- note removed: "Current per 100k Ohm Resitor Divider +3V3 / (100k + 100k) = 0.0165 mA Current per 200k Ohm Resistor Divider +3V3 / (200k + 200k) = 0.00825 mA Current per 10k Ohm Resitor Divider +3V3 / (10k + 10k) = 0.165 mA Current per 75k Load +3V3 / 75k = 0.044 mA Quiescent Current (Per Amplifier - 2x per chip) 7.5 mA Current Per TLV5616 1.1 mA"
Changed lines of the file:
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@@
 		)
 	)
-	(text "Current per 100k Ohm Resitor Divider\n+3V3 / (100k + 100k) = 0.0165 mA\n\nCurrent per 200k Ohm Resistor Divider\n+3V3 / (200k + 200k) = 0.00825 mA\n\nCurrent per 10k Ohm Resitor Divider\n+3V3 / (10k + 10k) = 0.165 mA\n\nCurrent per 75k Load\n+3V3 / 75k = 0.044 mA\n\nQuiescent Current (Per Amplifier - 2x per chip)\n7.5 mA\n\nCurrent Per TLV5616\n1.1 mA\n"
+	(text "Right Audio Current Consumption\n\nCurrent per 100k Ohm Resitor Divider\n+3V3 / (100k + 100k) = 0.0165 mA\n\nCurrent per 200k Ohm Resistor Divider\n+3V3 / (200k + 200k) = 0.00825 mA\n\nCurrent per 10k Ohm Resitor Divider\n+3V3 / (10k + 10k) = 0.165 mA\n\nCurrent per 75k Load\n+3V3 / 75k = 0.044 mA\n\nQuiescent Current (Per Amplifier - 2x per chip)\n7.5 mA\n\nCurrent Per TLV5616\n1.1 mA\n"
 		(exclude_from_sim no)
 		(at 118.745 155.575 0)

Commit message: PCB Layout
Parts:
- added R100, R101, R102, R103, R104, R96, R97, R98, R99: 2k, Resistor_SMD:R_0603_1608Metric_Pad0.98x0.95mm_HandSolder, symbol Device:R
- added R6: 0, Resistor_SMD:R_0603_1608Metric_Pad0.98x0.95mm_HandSolder, symbol Device:R
- added TP5: R_Treble, ECE445L:Testpoint_1x02_P2.54mm, symbol ECE445L:Testpoint
- added TP6: R_Mid, ECE445L:Testpoint_1x02_P2.54mm, symbol ECE445L:Testpoint
- added TP7: R_Bass, ECE445L:Testpoint_1x02_P2.54mm, symbol ECE445L:Testpoint
- Q1, Q2, Q3, Q4, Q5, Q6, Q7, Q8, Q9: value PZT2222A -> MMBF170; footprint Package_TO_SOT_SMD:SOT-223-3_TabPin2 -> Package_TO_SOT_SMD:SOT-23-3
Connections:
- net PB2: now also R100.1; no longer Q2.1 (B)
- net PB3: now also R101.2; no longer Q4.1 (B)
- net PB4: now also R98.1; no longer Q5.1 (B)
- net PB5: now also R99.2; no longer Q6.1 (B)
- net PB6: now also R96.1; no longer Q1.1 (B)
- net PB7: now also R97.2; no longer Q3.1 (B)
- net PC4: now also R102.1; no longer Q7.1 (B)
- net PC5: now also R103.1; no longer Q8.1 (B)
- net PC6: now also R104.1; no longer Q9.1 (B)
- net PD0: now also R6.1
- net R_Bass: now also R6.2, TP7.1 (A), TP7.2 (B)
- net R_Mid: now also TP6.1 (A), TP6.2 (B)
- net R_Treble: now also TP5.1 (A), TP5.2 (B)
- new net: Q6.1 (B), R99.1
- new net: Q1.1 (B), R96.2
- new net: Q7.1 (B), R102.2
- new net: Q5.1 (B), R98.2
- new net: Q3.1 (B), R97.1
- new net: Q8.1 (B), R103.2
- new net: Q2.1 (B), R100.2
- new net: Q4.1 (B), R101.1
- new net: Q9.1 (B), R104.2
Other:
- note added: "Optional Select for input to ADC"

Commit message: Pushing so i can work on my desktop
Other:
- note added: "Changed To MOSFETs (Had wrong part number)"
Changed lines of the file:
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@@
 		(comment 1 "Drawn By Ashton Knecht - atk836")
+	)
+	(text "Changed To MOSFETs\n(Had wrong part number)"
+		(exclude_from_sim no)
+		(at 259.715 162.56 0)
+		(effects
+			(font
+				(size 1.27 1.27)
+			)
+		)
 	)
 	(text "Variable Gain"
 		(exclude_from_sim no)
 		(at 66.675 62.865 0)
+		(effects
+			(font
+				(size 1.27 1.27)
+			)
+		)
+	)
+	(text "Changed To MOSFETs\n(Had wrong part number)"
+		(exclude_from_sim no)
+		(at 40.005 77.47 0)
 		(effects
 			(font
@@
 		(exclude_from_sim no)
 		(at 100.965 78.74 0)
+		(effects
+			(font
+				(size 1.27 1.27)
+			)
+		)
+	)
+	(text "Changed To MOSFETs\n(Had wrong part number)"
+		(exclude_from_sim no)
+		(at 80.645 128.905 0)
 		(effects
 			(font
@@
 		(effects
 			(font
+				(size 1.27 1.27)
+			)
+		)
+	)
+	(text "Changed To MOSFETs\n(Had wrong part number)"
+		(exclude_from_sim no)
+		(at 40.005 192.405 0)
+		(effects
+			(font

Commit message: Final PCB commit
Parts:
- removed Q7, Q8, Q9: MMBF170, Package_TO_SOT_SMD:SOT-23-3, symbol Transistor_BJT:PZT2222A
- removed R102, R103, R104: 2k, Resistor_SMD:R_0603_1608Metric_Pad0.98x0.95mm_HandSolder, symbol Device:R
- removed R32, R34, R35, R36, R38: 100k, Resistor_SMD:R_0603_1608Metric_Pad0.98x0.95mm_HandSolder, symbol Device:R
- removed R37: 75K, Resistor_SMD:R_0603_1608Metric_Pad0.98x0.95mm_HandSolder, symbol Device:R
- Q1, Q2, Q3, Q4, Q5, Q6: footprint Package_TO_SOT_SMD:SOT-23-3 -> Package_TO_SOT_SMD:SOT-23; symbol Transistor_BJT:PZT2222A -> Transistor_FET:MMBF170
- R14: renamed from R10; value 100k -> 184k
- R15: renamed from R11; value 100k -> 68.8k
- R16: renamed from R12; value 20k -> 40k
- R17: renamed from R13; value 20k -> 40k
- R18: renamed from R14; value 10k -> 30k
- R19: renamed from R15; value 10k -> 30k
- R25: renamed from R18; value 100k -> 184k
- R26: renamed from R19; value 100k -> 68.8k
- R28: renamed from R20; value 20k -> 40k
- R30: renamed from R21; value 10k -> 30k
- R41: renamed from R33; value 100k -> 50k
- renumbered C21 to C10, C22 to C11, C23 to C12, C24 to C13, C25 to C14, C26 to C15, C15 to C4, C16 to C5, C17 to C6, C18 to C7, C19 to C8, C20 to C9, R8 to R10, R96 to R11, R9 to R12, R100 to R13, R16 to R20, R17 to R21, R97 to R22, R101 to R23, R98 to R24, R6 to R27, R23 to R29, R22 to R31, R99 to R32, R24 to R33, R25 to R34, R26 to R35, R27 to R36, R28 to R37, R29 to R38, R30 to R39, R31 to R40, R7 to R9, TP5 to TP7, TP6 to TP8, TP7 to TP9, U6 to U5, U7 to U6, U8 to U7, U9 to U8, U10 to U9
Connections:
- net GND: now also Q1.2 (S), Q2.2 (S), Q3.2 (S), Q4.2 (S), Q5.2 (S), Q6.2 (S); no longer Q1.3 (E), Q2.3 (E), Q3.3 (E), Q4.3 (E), Q5.3 (E), Q6.3 (E)
- net R_AudioOut: no longer U8.7
- net at R30.1: now also Q6.3 (D); no longer Q6.2 (C)
- net at R28.2: now also Q5.3 (D); no longer Q5.2 (C)
- net at R17.2: now also Q2.3 (D); no longer Q2.2 (C)
- net at U8.5 (+): now also C14.2, R39.1, R40.2
- net at R18.1: now also Q3.3 (D); no longer Q3.2 (C)
- net at R19.1: now also Q4.3 (D); no longer Q4.2 (C)
- net at R16.2: now also Q1.3 (D); no longer Q1.2 (C)
- new net R_AudioBuf: R41.1, U8.7
Other:
- moved on the sheet: R35, R36, R37, R38, R39, R40, R41, U8A, U8B
