File: hw/ECE445L_Lab7/Lab7_microcontroller.kicad_sch (KiCad schematic)
At the start: 6 parts, among them J2 EK-TM4C123GXL, U3 ESP32-D0WD-V3, U5 FT232R

Commit message: Pushing so i can work on my desktop
Connections:
- net +3V3: now also U3.15 (1EN); no longer U3.1 (EN)
- net +VRail: now also U3.1 (VIN); no longer U3.15 (VIN)
- net ESP_IN_USB_OUT: now also U3.22 (GPIO17); no longer U3.24 (GPIO17)
- net ESP_OUT_USB_IN: now also U3.21 (GPIO16); no longer U3.25 (GPIO16)
- net GND: now also U3.17 (GND), U3.2 (GND); no longer U3.14 (GND), U3.29 (GND)
- net LAUDIO_CLK: now also U3.3 (GPIO13); no longer U3.13 (GPIO13)
- net LAUDIO_FS: now also U3.5 (GPIO14); no longer U3.11 (GPIO14)
- net LAUDIO_OUT: now also U3.4 (GPIO12); no longer U3.12 (GPIO12)
- net PB0: now also U3.28 (GPIO1); no longer U3.18 (GPIO1)
- net PB1: now also U3.27 (GPIO3); no longer U3.19 (GPIO3)
- net RAUDIO_CLK: now also U3.7 (GPIO26); no longer U3.9 (GPIO26)
- net RAUDIO_FS: now also U3.6 (GPIO27); no longer U3.10 (GPIO27)

Commit message: Final PCB commit
Parts:
- removed U5: FT232R, symbol ECE445L:FT232R-Breakout
- added U4: FT232R, ECE445L:FT232R-Breakout, symbol ECE445L:FT232R-Breakout
- renumbered R114 to R6, R115 to R7, R116 to R8
Connections:
- net ESP_IN_USB_OUT: now also U4.2 (TXD)
- net ESP_OUT_USB_IN: now also U4.3 (RXD)
- net GND: now also U4.4 (GND)
- net at R6.2: now also U4.1 (3V3)
Other:
- note added: "Please note that the ESP we are using doesn't have USB We have used interfaced the FT2322R and ESP in unit testing"
- moved on the sheet: R6
